Commit message: Add launch option to load velodyne.
Signed-off-by: Jelmer de Wolde <jelmer.de.wolde@alliander.com>

File: ros2_ws/src/rcdt_panther/urdf/panther.urdf.xacro (robot description, xacro)
@@ -16,7 +16,10 @@
     battery_config_file="" />
   <!-- Load Velodyne: -->
-  <xacro:include filename="$(find rcdt_sensors)/urdf/rcdt_velodyne.urdf.xacro" />
-  <xacro:VLP-16>
-    <origin xyz="0.18 0 0.03" rpy="0 0 0" />
-  </xacro:VLP-16>
+  <xacro:arg name="load_velodyne" default="false" />
+  <xacro:if value="$(arg load_velodyne)">
+    <xacro:include filename="$(find rcdt_sensors)/urdf/rcdt_velodyne.urdf.xacro" />
+    <xacro:VLP-16>
+      <origin xyz="0.18 0 0.03" rpy="0 0 0" />
+    </xacro:VLP-16>
+  </xacro:if>
 </robot>
