Commit message: Update urdf to 2.2.1
Signed-off-by: Jelmer de Wolde <jelmer.de.wolde@alliander.com>

File: ros2_ws/src/rcdt_gazebo/urdf/remappings.urdf.xacro (robot description, xacro)
@@ -14,10 +14,13 @@
     <!-- NONE -->
     <!-- panther: -->
+    <remapping>drive_controller/cmd_vel_unstamped:=cmd_vel</remapping>
+    <remapping>drive_controller/odom:=odometry/wheels</remapping>
+    <remapping>drive_controller/transition_event:=drive_controller/_transition_event</remapping>
     <remapping>gz_ros2_control/e_stop:=hardware/e_stop</remapping>
     <remapping>gz_ros2_control/e_stop_reset:=hardware/e_stop_reset</remapping>
     <remapping>gz_ros2_control/e_stop_trigger:=hardware/e_stop_trigger</remapping>
     <remapping>imu_broadcaster/imu:=imu/data</remapping>
-    <remapping>drive_controller/cmd_vel_unstamped:=cmd_vel</remapping>
-    <remapping>drive_controller/odom:=odometry/wheels</remapping>
+    <remapping>imu_broadcaster/transition_event:=imu_broadcaster/_transition_event</remapping>
+    <remapping>joint_state_broadcaster/transition_event:=joint_state_broadcaster/_transition_event</remapping>
   </xacro:macro>
 </robot>

File: ros2_ws/src/rcdt_panther/urdf/adapted/gazebo.urdf.xacro (robot description, xacro)
@@ -117,5 +117,5 @@
   <xacro:macro name="light" params="reference_frame name topic namespace:=''">
     <gazebo>
-      <plugin filename="LEDStrip" name="panther_gazebo::LEDStrip">
+      <plugin filename="LEDStrip" name="husarion_ugv_gazebo::LEDStrip">
         <light_name>${name}</light_name>
         <topic>${topic}</topic>

File: ros2_ws/src/rcdt_panther/urdf/adapted/panther_macro.urdf.xacro (robot description, xacro)
@@ -10,6 +10,5 @@
   <xacro:macro
     name="panther_robot"
-    params="panther_version
-            wheel_config_file
+    params="wheel_config_file
             controller_config_file
             battery_config_file
@@ -19,6 +18,4 @@
             namespace:=''
             connected_to:=''">
-    <!-- Map params to args: -->
-    <xacro:arg name="use_sim" default="${use_sim}" />
     <xacro:if value="${use_sim}">
       <xacro:property name="imu_xyz" value="-0.195 0.010 0.085" />
@@ -27,9 +24,10 @@
     <xacro:property name="ns" value='${namespace + "/" if namespace else ""}' />
     <xacro:property name="wheel_config" value="${xacro.load_yaml(wheel_config_file)}" />
-    <xacro:property name="wheel_separation_x" value="0.44" />
+    <xacro:property name="wheelbase" value="0.44" />
+    <xacro:property name="wheel_mount_point_y" value="0.2575" />
     <!-- INCLUDE ROBOT PARTS DEFINITIONS -->
-    <xacro:include filename="$(find panther_description)/urdf/body.urdf.xacro" ns="body" />
+    <xacro:include filename="$(find husarion_ugv_description)/urdf/panther/base.urdf.xacro" ns="body" />
     <xacro:include filename="$(find rcdt_panther)/urdf/adapted/gazebo.urdf.xacro" ns="gazebo" />
-    <xacro:include filename="$(find panther_description)/urdf/wheel.urdf.xacro" ns="wheel" />
+    <xacro:include filename="$(find husarion_ugv_description)/urdf/common/wheel.urdf.xacro" ns="wheel" />
     <!-- BODY DECLARATION -->
     <xacro:body.body
@@ -39,28 +37,31 @@
     <!-- WHEEL DECLARATION -->
     <xacro:wheel.wheel
-      wheel_config="${wheel_config}"
-      wheel_separation_x="${wheel_separation_x}"
+      config="${wheel_config}"
+      mount_point_x="${wheelbase/2.0}"
+      mount_point_y="${wheel_mount_point_y}"
       prefix="fl" />
     <xacro:wheel.wheel
-      wheel_config="${wheel_config}"
-      wheel_separation_x="${wheel_separation_x}"
+      config="${wheel_config}"
+      mount_point_x="${wheelbase/2.0}"
+      mount_point_y="${wheel_mount_point_y}"
       prefix="fr" />
     <xacro:wheel.wheel
-      wheel_config="${wheel_config}"
-      wheel_separation_x="${wheel_separation_x}"
+      config="${wheel_config}"
+      mount_point_x="${wheelbase/2.0}"
+      mount_point_y="${wheel_mount_point_y}"
       prefix="rl" />
     <xacro:wheel.wheel
-      wheel_config="${wheel_config}"
-      wheel_separation_x="${wheel_separation_x}"
+      config="${wheel_config}"
+      mount_point_x="${wheelbase/2.0}"
+      mount_point_y="${wheel_mount_point_y}"
       prefix="rr" />
     <ros2_control name="${ns}panther_system" type="system">
       <hardware>
         <xacro:if value="${use_sim}">
-          <plugin>panther_gazebo/GzPantherSystem</plugin>
+          <plugin>husarion_ugv_gazebo/EStopSystem</plugin>
           <param name="e_stop_initial_state">true</param>
         </xacro:if>
-        <xacro:unless value="$(arg use_sim)">
-          <plugin>panther_hardware_interfaces/PantherSystem</plugin>
-          <param name="panther_version">${panther_version}</param>
+        <xacro:unless value="${use_sim}">
+          <plugin>husarion_ugv_hardware_interfaces/PantherSystem</plugin>
           <param name="encoder_resolution">1600</param>
           <param name="gear_ratio">30.08</param>
@@ -70,5 +71,5 @@
           <!-- Max RPM speed set in the Roboteq driver (MXRPM parameter) -->
           <param name="max_rpm_motor_speed">3600.0</param>
-          <param name="can_interface_name">panther_can</param>
+          <param name="can_interface_name">robot_can</param>
           <param name="master_can_id">3</param>
           <param name="front_driver_can_id">1</param>
@@ -129,8 +130,8 @@
       </xacro:if>
     </ros2_control>
-    <xacro:unless value="$(arg use_sim)">
+    <xacro:unless value="${use_sim}">
       <ros2_control name="${ns}imu" type="sensor">
         <hardware>
-          <plugin>panther_hardware_interfaces/PantherImuSensor</plugin>
+          <plugin>husarion_ugv_hardware_interfaces/PhidgetImuSensor</plugin>
           <param name="serial">-1</param>
           <param name="hub_port">0</param>

File: ros2_ws/src/rcdt_panther/urdf/original/gazebo.urdf.xacro (robot description, xacro)
@@ -34,10 +34,13 @@
         <ros>
           <namespace>${namespace}</namespace>
+          <remapping>drive_controller/cmd_vel_unstamped:=cmd_vel</remapping>
+          <remapping>drive_controller/odom:=odometry/wheels</remapping>
+          <remapping>drive_controller/transition_event:=drive_controller/_transition_event</remapping>
           <remapping>gz_ros2_control/e_stop:=hardware/e_stop</remapping>
           <remapping>gz_ros2_control/e_stop_reset:=hardware/e_stop_reset</remapping>
           <remapping>gz_ros2_control/e_stop_trigger:=hardware/e_stop_trigger</remapping>
           <remapping>imu_broadcaster/imu:=imu/data</remapping>
-          <remapping>drive_controller/cmd_vel_unstamped:=cmd_vel</remapping>
-          <remapping>drive_controller/odom:=odometry/wheels</remapping>
+          <remapping>imu_broadcaster/transition_event:=imu_broadcaster/_transition_event</remapping>
+          <remapping>joint_state_broadcaster/transition_event:=joint_state_broadcaster/_transition_event</remapping>
         </ros>
       </plugin>
@@ -101,5 +104,5 @@
   <xacro:macro name="light" params="reference_frame name topic namespace:=''">
     <gazebo>
-      <plugin filename="LEDStrip" name="panther_gazebo::LEDStrip">
+      <plugin filename="LEDStrip" name="husarion_ugv_gazebo::LEDStrip">
         <light_name>${name}</light_name>
         <topic>${topic}</topic>

File: ros2_ws/src/rcdt_panther/urdf/original/panther_macro.urdf.xacro (robot description, xacro)
@@ -3,6 +3,5 @@
   <xacro:macro
     name="panther_robot"
-    params="panther_version
-            wheel_config_file
+    params="wheel_config_file
             controller_config_file
             battery_config_file
@@ -17,9 +16,10 @@
     <xacro:property name="ns" value='${namespace + "/" if namespace else ""}' />
     <xacro:property name="wheel_config" value="${xacro.load_yaml(wheel_config_file)}" />
-    <xacro:property name="wheel_separation_x" value="0.44" />
+    <xacro:property name="wheelbase" value="0.44" />
+    <xacro:property name="wheel_mount_point_y" value="0.2575" />
     <!-- INCLUDE ROBOT PARTS DEFINITIONS -->
-    <xacro:include filename="$(find panther_description)/urdf/body.urdf.xacro" ns="body" />
-    <xacro:include filename="$(find panther_description)/urdf/gazebo.urdf.xacro" ns="gazebo" />
-    <xacro:include filename="$(find panther_description)/urdf/wheel.urdf.xacro" ns="wheel" />
+    <xacro:include filename="$(find husarion_ugv_description)/urdf/panther/base.urdf.xacro" ns="body" />
+    <xacro:include filename="$(find husarion_ugv_description)/urdf/common/gazebo.urdf.xacro" ns="gazebo" />
+    <xacro:include filename="$(find husarion_ugv_description)/urdf/common/wheel.urdf.xacro" ns="wheel" />
     <!-- BODY DECLARATION -->
     <xacro:body.body
@@ -29,28 +29,31 @@
     <!-- WHEEL DECLARATION -->
     <xacro:wheel.wheel
-      wheel_config="${wheel_config}"
-      wheel_separation_x="${wheel_separation_x}"
+      config="${wheel_config}"
+      mount_point_x="${wheelbase/2.0}"
+      mount_point_y="${wheel_mount_point_y}"
       prefix="fl" />
     <xacro:wheel.wheel
-      wheel_config="${wheel_config}"
-      wheel_separation_x="${wheel_separation_x}"
+      config="${wheel_config}"
+      mount_point_x="${wheelbase/2.0}"
+      mount_point_y="${wheel_mount_point_y}"
       prefix="fr" />
     <xacro:wheel.wheel
-      wheel_config="${wheel_config}"
-      wheel_separation_x="${wheel_separation_x}"
+      config="${wheel_config}"
+      mount_point_x="${wheelbase/2.0}"
+      mount_point_y="${wheel_mount_point_y}"
       prefix="rl" />
     <xacro:wheel.wheel
-      wheel_config="${wheel_config}"
-      wheel_separation_x="${wheel_separation_x}"
+      config="${wheel_config}"
+      mount_point_x="${wheelbase/2.0}"
+      mount_point_y="${wheel_mount_point_y}"
       prefix="rr" />
     <ros2_control name="${ns}panther_system" type="system">
       <hardware>
         <xacro:if value="${use_sim}">
-          <plugin>panther_gazebo/GzPantherSystem</plugin>
+          <plugin>husarion_ugv_gazebo/EStopSystem</plugin>
           <param name="e_stop_initial_state">true</param>
         </xacro:if>
-        <xacro:unless value="$(arg use_sim)">
-          <plugin>panther_hardware_interfaces/PantherSystem</plugin>
-          <param name="panther_version">${panther_version}</param>
+        <xacro:unless value="${use_sim}">
+          <plugin>husarion_ugv_hardware_interfaces/PantherSystem</plugin>
           <param name="encoder_resolution">1600</param>
           <param name="gear_ratio">30.08</param>
@@ -60,5 +63,5 @@
           <!-- Max RPM speed set in the Roboteq driver (MXRPM parameter) -->
           <param name="max_rpm_motor_speed">3600.0</param>
-          <param name="can_interface_name">panther_can</param>
+          <param name="can_interface_name">robot_can</param>
           <param name="master_can_id">3</param>
           <param name="front_driver_can_id">1</param>
@@ -119,8 +122,8 @@
       </xacro:if>
     </ros2_control>
-    <xacro:unless value="$(arg use_sim)">
+    <xacro:unless value="${use_sim}">
       <ros2_control name="${ns}imu" type="sensor">
         <hardware>
-          <plugin>panther_hardware_interfaces/PantherImuSensor</plugin>
+          <plugin>husarion_ugv_hardware_interfaces/PhidgetImuSensor</plugin>
           <param name="serial">-1</param>
           <param name="hub_port">0</param>

File: ros2_ws/src/rcdt_panther/urdf/panther.urdf.xacro (robot description, xacro)
@@ -9,8 +9,7 @@
   <xacro:arg name="connected_to" default="" />
   <!-- Load panther: -->
-  <xacro:include filename="$(find husarion_ugv_description)/urdf/panther/panther_macro.urdf.xacro"
+  <xacro:include filename="$(find rcdt_panther)/urdf/adapted/panther_macro.urdf.xacro"
     ns="husarion" />
   <xacro:husarion.panther_robot
-    panther_version="1.0"
     use_sim="$(arg simulation)"
     wheel_config_file="$(find husarion_ugv_description)/config/WH01.yaml"
