Commit message: Add ZED2i mesh and update URDF references to use the new mesh path
Signed-off-by: Max Waterhout <max.waterhout@hotmail.nl>

File: ros2_ws/src/rcdt_sensors/urdf/zed_macro.urdf.xacro (robot description, xacro)
@@ -105,5 +105,5 @@
           <origin xyz="${screw_offset_x} 0 ${screw_offset_z}" rpy="0 0 0"/>
           <geometry>
-<mesh filename="file://$(find zed_msgs)/meshes/${model}.stl"/>
+<mesh filename="file://$(find rcdt_sensors)/meshes/${model}.stl"/>
           </geometry>
           <material name="${model}_mat" />
@@ -112,5 +112,5 @@
           <origin xyz="${screw_offset_x} 0 ${screw_offset_z}" rpy="0 0 0"/>
           <geometry>
-<mesh filename="file://$(find zed_msgs)/meshes/${model}.stl"/>
+<mesh filename="file://$(find rcdt_sensors)/meshes/${model}.stl"/>
           </geometry>
         </collision>
@@ -129,5 +129,5 @@
             <origin xyz="0 0 0" rpy="0 0 0"/>
             <geometry>
-  <mesh filename="file://$(find zed_msgs)/meshes/${model}.stl"/>
+  <mesh filename="file://$(find rcdt_sensors)/meshes/${model}.stl"/>
             </geometry>
             <material name="${model}_mat" />
@@ -136,5 +136,5 @@
             <origin xyz="0 0 0" rpy="0 0 0"/>
             <geometry>
-  <mesh filename="file://$(find zed_msgs)/meshes/${model}.stl"/>
+  <mesh filename="file://$(find rcdt_sensors)/meshes/${model}.stl"/>
             </geometry>
           </collision>
@@ -158,5 +158,5 @@
             <origin xyz="0 0 0" rpy="0 0 0"/>
             <geometry>
-  <mesh filename="file://$(find zed_msgs)/meshes/${model}.stl"/>
+  <mesh filename="file://$(find rcdt_sensors)/meshes/${model}.stl"/>
             </geometry>
             <material name="${model}_mat" />
@@ -165,5 +165,5 @@
             <origin xyz="0 0 0" rpy="0 0 0"/>
             <geometry>
-  <mesh filename="file://$(find zed_msgs)/meshes/${model}.stl"/>
+  <mesh filename="file://$(find rcdt_sensors)/meshes/${model}.stl"/>
             </geometry>
           </collision>
