Commit message: Fix for use on real robot.
Signed-off-by: Jelmer de Wolde <jelmer.de.wolde@alliander.com>

File: ros2_ws/src/rcdt_sensors/urdf/rcdt_velodyne.urdf.xacro (robot description, xacro)
@@ -7,5 +7,5 @@
 Based on:
 1.https://bitbucket.org/DataspeedInc/velodyne_simulator/src/master/velodyne_description/urdf/VLP-16.urdf.xacro
-2.https://github.com/husarion/ros_components_description/blob/ros2/urdf/velodyne_puck.urdf.xacro
+2.https://github.com/husarion/husarion_components_description/blob/ros2/urdf/velodyne_puck.urdf.xacro
 -->
 <robot xmlns:xacro="http://www.ros.org/wiki/xacro" name="VLP-16">
@@ -15,4 +15,5 @@
     *origin
     namespace
+    name:=velodyne
     update_rate:=10
     lasers:=16
@@ -51,7 +52,7 @@
       <origin xyz="0 0 0.0377" rpy="0 0 0" />
       <parent link="base_link" />
-      <child link="lidar" />
+      <child link="${name}" />
     </joint>
-    <link name="lidar">
+    <link name="${name}">
       <inertial>
         <mass value="0.01" />
@@ -66,5 +67,5 @@
       </visual>
     </link>
-    <gazebo reference="lidar">
+    <gazebo reference="${name}">
       <sensor type="gpu_lidar" name="${namespace}">
         <always_on>true</always_on>
@@ -72,6 +73,6 @@
         <topic>${namespace}/scan</topic>
         <visualize>false</visualize>
-        <gz_frame_id>${namespace}/lidar</gz_frame_id>
-        <frame_id>${namespace}/lidar</frame_id>
+        <gz_frame_id>${namespace}/${name}</gz_frame_id>
+        <frame_id>${namespace}/${name}</frame_id>
         <ray>
           <scan>

Commit message: Add lidar support.
Signed-off-by: Jelmer de Wolde <jelmer.de.wolde@alliander.com>

File: ros2_ws/src/rcdt_sensors/urdf/rcdt_velodyne.urdf.xacro (robot description, xacro)
@@ -15,4 +15,5 @@
     *origin
     namespace
+    parent
     name:=velodyne
     update_rate:=10
@@ -67,4 +68,14 @@
       </visual>
     </link>
+    <!-- Gazebo requires a joint to a link called "world" for statically mounted robots -->
+    <xacro:if value="${parent != ''}">
+      <xacro:if value="${parent == 'world'}">
+        <link name="${parent}" />
+        <joint name="${parent}_joint" type="fixed">
+          <parent link="${parent}" />
+          <child link="base_link" />
+        </joint>
+      </xacro:if>
+    </xacro:if>
     <gazebo reference="${name}">
       <sensor type="gpu_lidar" name="${namespace}">
@@ -104,5 +115,5 @@
     </gazebo>
   </xacro:macro>
-  <xacro:VLP-16 namespace="velodyne">
+  <xacro:VLP-16 namespace="$(arg namespace)" parent="$(arg parent)">
     <origin xyz="0 0 0" rpy="0 0 0" />
   </xacro:VLP-16>

Commit message: WIP
Signed-off-by: Jelmer de Wolde <jelmer.de.wolde@alliander.com>

File: ros2_ws/src/rcdt_sensors/urdf/rcdt_velodyne.urdf.xacro (robot description, xacro)
@@ -15,4 +15,5 @@
     *origin
     namespace
+    parent
     name:=velodyne
     update_rate:=10
@@ -67,4 +68,14 @@
       </visual>
     </link>
+    <!-- Gazebo requires a joint to a link called "world" for statically mounted robots -->
+    <xacro:if value="${parent != ''}">
+      <xacro:if value="${parent == 'world'}">
+        <link name="${parent}" />
+        <joint name="${parent}_joint" type="fixed">
+          <parent link="${parent}" />
+          <child link="base_link" />
+        </joint>
+      </xacro:if>
+    </xacro:if>
     <gazebo reference="${name}">
       <sensor type="gpu_lidar" name="${namespace}">
@@ -104,5 +115,7 @@
     </gazebo>
   </xacro:macro>
-  <xacro:VLP-16 namespace="velodyne">
+  <xacro:arg name="namespace" default="" />
+  <xacro:arg name="parent" default="" />
+  <xacro:VLP-16 namespace="$(arg namespace)" parent="$(arg parent)">
     <origin xyz="0 0 0" rpy="0 0 0" />
   </xacro:VLP-16>
