Commit message: Introduce calibration method.
Signed-off-by: Jelmer de Wolde <jelmer.de.wolde@alliander.com>

File: ros2_ws/src/rcdt_sensors/urdf/rcdt_realsense_d435.urdf.xacro (robot description, xacro)
@@ -21,5 +21,5 @@
       parent="${parent}"
       use_nominal_extrinsics="true">
-      <origin xyz="0 0.015 0" rpy="0 0 0" />
+      <origin xyz="0 0 0" rpy="0 0 0" />
     </xacro:sensor_d435>
     <!-- Add gazebo plugin: -->
@@ -59,5 +59,5 @@
             </image>
             <clip>
-              <near>0.01</near>
+              <near>0.1</near>
               <far>65.536</far>
             </clip>

Commit message: Improve camera position, use low res in simulation to avoid depth camera display offset.
Signed-off-by: Jelmer de Wolde <jelmer.de.wolde@alliander.com>

File: ros2_ws/src/rcdt_sensors/urdf/rcdt_realsense_d435.urdf.xacro (robot description, xacro)
@@ -21,5 +21,5 @@
       parent="${parent}"
       use_nominal_extrinsics="true">
-      <origin xyz="0 0.015 0" rpy="0 0 0" />
+      <origin xyz="0 0 0" rpy="0 0 0" />
     </xacro:sensor_d435>
     <!-- Add gazebo plugin: -->
@@ -36,6 +36,6 @@
             <horizontal_fov>${69.0/180.0*pi}</horizontal_fov>
             <image>
-              <width>640</width>
-              <height>480</height>
+              <width>320</width>
+              <height>240</height>
             </image>
             <clip>
@@ -55,6 +55,6 @@
             <horizontal_fov>${69.0/180.0*pi}</horizontal_fov> <!-- Using color FOV, to avoid align. -->
             <image>
-              <width>640</width>
-              <height>480</height>
+              <width>320</width>
+              <height>240</height>
             </image>
             <clip>

Commit message: Add realsense to modular system.
Signed-off-by: Jelmer de Wolde <jelmer.de.wolde@alliander.com>

File: ros2_ws/src/rcdt_sensors/urdf/rcdt_realsense_d435.urdf.xacro (robot description, xacro)
@@ -7,20 +7,26 @@
   <xacro:macro name="rcdt_realsense_d435"
     params="
-    robot_namespace
-    device_namespace
+    namespace
+    parent
     name:=camera
     gazebo:=true
-    parent:=world
     align:=color
     ">
-    <!-- Create world link if this is the parent: -->
-    <xacro:if value="${parent == 'world'}">
-      <link name="${parent}" />
+    <!-- Gazebo requires a joint to a link called "world" for statically mounted robots -->
+    <xacro:if value="${parent != ''}">
+      <xacro:if value="${parent == 'world'}">
+        <link name="${parent}" />
+        <joint name="${parent}_joint" type="fixed">
+          <parent link="${parent}" />
+          <child link="base_link" />
+        </joint>
+      </xacro:if>
     </xacro:if>
     <!-- Include realsense xacro: -->
+    <link name="base_link" />
     <xacro:include filename="$(find realsense2_description)/urdf/_d435.urdf.xacro" />
     <xacro:sensor_d435
-      name="${device_namespace}/${name}"
-      parent="${parent}"
+      name="${name}"
+      parent="base_link"
       use_nominal_extrinsics="true">
       <origin xyz="0 0 0" rpy="0 0 0" />
@@ -28,20 +34,20 @@
     <!-- Add gazebo plugin: -->
     <xacro:if value="${gazebo}">
-      <gazebo reference="${device_namespace}/${name}_${align}_frame">
+      <gazebo reference="${name}_${align}_frame">
         <!-- rgb_camera: -->
         <sensor type="camera" name="intel_realsense_d435_color">
           <always_on>true</always_on>
           <update_rate>30.0</update_rate>
-          <topic>${robot_namespace}/${device_namespace}/color/image_raw</topic>
+          <topic>${namespace}/color/image_raw</topic>
           <visualize>false</visualize>
-          <gz_frame_id>${robot_namespace}/${device_namespace}/${name}_${align}_optical_frame</gz_frame_id>
+          <gz_frame_id>${namespace}/${name}_${align}_optical_frame</gz_frame_id>
           <camera>
             <horizontal_fov>${69.0/180.0*pi}</horizontal_fov>
             <image>
-              <width>320</width>
-              <height>240</height>
+              <width>640</width>
+              <height>480</height>
             </image>
             <clip>
-              <near>0.02</near>
+              <near>0.1</near>
               <far>300.0</far>
             </clip>
@@ -52,15 +58,15 @@
           <always_on>true</always_on>
           <update_rate>30.0</update_rate>
-          <topic>${robot_namespace}/${device_namespace}/depth/image_rect_raw_float</topic>
+          <topic>${namespace}/depth/image_rect_raw_float</topic>
           <visualize>false</visualize>
-          <gz_frame_id>${robot_namespace}/${device_namespace}/${name}_${align}_optical_frame</gz_frame_id>
+          <gz_frame_id>${namespace}/${name}_${align}_optical_frame</gz_frame_id>
           <camera>
             <horizontal_fov>${69.0/180.0*pi}</horizontal_fov> <!-- Using color FOV, to avoid align. -->
             <image>
-              <width>320</width>
-              <height>240</height>
+              <width>640</width>
+              <height>480</height>
             </image>
             <clip>
-              <near>0.01</near>
+              <near>0.2</near>
               <far>65.536</far>
             </clip>
@@ -70,3 +76,6 @@
     </xacro:if>
   </xacro:macro>
+  <xacro:arg name="namespace" default="realsense" />
+  <xacro:arg name="parent" default="" />
+  <xacro:rcdt_realsense_d435 namespace="$(arg namespace)" parent="$(arg parent)"/>
 </robot>
