Commit message: Fix zed xacro for simulation.
Signed-off-by: Jelmer de Wolde <jelmer.de.wolde@alliander.com>

File: ros2_ws/src/rcdt_sensors/urdf/rcdt_zed2i.urdf.xacro (robot description, xacro)
@@ -6,48 +6,92 @@
 <robot xmlns:xacro="http://www.ros.org/wiki/xacro" name="rcdt_zed2i">
   <xacro:macro name="rcdt_zed2i"
-               params="robot_namespace
-                       device_namespace
-                       parent:=world
-                       model:=zed2i
-                       enable_gnss:=false
-                       xyz:='0 0 0' rpy:='0 0 0' ">
-    <xacro:include filename="$(find zed_wrapper)/urdf/zed_macro.urdf.xacro"/>
-    <xacro:zed_camera name="${device_namespace}"
-                      model="${model}"
-                      enable_gnss="${enable_gnss}">
-      <origin xyz="${xyz}" rpy="${rpy}"/>
+    params="
+    namespace
+    parent:=world
+    name:=camera
+    gazebo:=true
+    model:=zed2i
+    enable_gnss:=false
+    align:=left
+    xyz:='0 0 0'
+    rpy:='0 0 0'
+    ">
+    <!-- Gazebo requires a joint to a link called "world" for statically mounted robots -->
+    <xacro:if value="${parent != ''}">
+      <xacro:if value="${parent == 'world'}">
+        <link name="${parent}" />
+        <joint name="${parent}_joint" type="fixed">
+          <parent link="${parent}" />
+          <child link="base_link" />
+        </joint>
+      </xacro:if>
+    </xacro:if>
+    <!-- Gazebo requires a base link with inertia: -->
+    <link name="base_link">
+      <inertial>
+        <mass value="0.01" />
+        <origin xyz="0 0 0" />
+        <inertia ixx="1e-7" ixy="0" ixz="0" iyy="1e-7" iyz="0" izz="1e-7" />
+      </inertial>
+    </link>
+    <joint name="base_joint" type="fixed">
+      <origin xyz="0 0 0" rpy="0 0 0" />
+      <parent link="base_link" />
+      <child link="${namespace}_camera_link" />
+    </joint>
+    <!-- Include zed xacro: -->
+    <xacro:include filename="$(find zed_wrapper)/urdf/zed_macro.urdf.xacro" />
+    <xacro:zed_camera
+      name="${namespace}"
+      model="${model}"
+      enable_gnss="${enable_gnss}">
+      <origin xyz="${xyz}" rpy="${rpy}" />
     </xacro:zed_camera>
-    <gazebo reference="${device_namespace}_left_camera_frame">
-      <sensor type="camera" name="${device_namespace}_rgb">
-        <!-- Shift the lens 1 cm forward in +X (robot-forward) -->
-        <pose>0.01 0 0  0 0 0</pose>
-        <always_on>true</always_on>
-        <update_rate>30.0</update_rate>
-        <topic>/zed/zed_node/rgb/image_rect_color</topic>
-        <visualize>false</visualize>
-        <camera>
-          <horizontal_fov>1.204277</horizontal_fov>
-          <image><width>640</width><height>360</height></image>
-          <clip><near>0.02</near><far>300.0</far></clip>
-        </camera>
-      </sensor>
-    </gazebo>
-    <gazebo reference="${device_namespace}_left_camera_frame">
-      <sensor type="depth_camera" name="${device_namespace}_depth">
-      <pose>0.01 0 0  0 0 0</pose>
-      <always_on>true</always_on>
-      <update_rate>30.0</update_rate>
-      <topic>/zed/zed_node/depth/depth_registered</topic>
-      <visualize>false</visualize>
-      <camera>
-        <horizontal_fov>1.204277</horizontal_fov>
-        <image><width>640</width><height>360</height></image>
-        <clip>
-          <near>0.01</near>
-          <far>65.536</far>
-        </clip>
-      </camera>
-      </sensor>
-    </gazebo>
+    <!-- Add gazebo plugin: -->
+    <xacro:if value="${gazebo}">
+      <gazebo reference="${namespace}_${align}_camera_frame">
+        <!-- rgb_camera: -->
+        <sensor type="camera" name="zed2i_color">
+          <always_on>true</always_on>
+          <update_rate>30.0</update_rate>
+          <topic>${namespace}/color/image_raw</topic>
+          <visualize>false</visualize>
+          <gz_frame_id>${namespace}/${namespace}_${align}_camera_optical_frame</gz_frame_id>
+          <camera>
+            <horizontal_fov>${110.0/180.0*pi}</horizontal_fov>
+            <image>
+              <width>640</width>
+              <height>480</height>
+            </image>
+            <clip>
+              <near>0.1</near>
+              <far>300.0</far>
+            </clip>
+          </camera>
+        </sensor>
+        <!-- depth camera -->
+        <sensor type="depth_camera" name="zed2i_depth">
+          <always_on>true</always_on>
+          <update_rate>30.0</update_rate>
+          <topic>${namespace}/depth/image_rect_raw_float</topic>
+          <visualize>false</visualize>
+          <gz_frame_id>${namespace}/${namespace}_${align}_camera_optical_frame</gz_frame_id>
+          <camera>
+            <horizontal_fov>${110.0/180.0*pi}</horizontal_fov>
+            <image>
+              <width>640</width>
+              <height>480</height>
+            </image>
+            <clip>
+              <near>0.2</near>
+              <far>65.536</far>
+            </clip>
+          </camera>
+        </sensor>
+      </gazebo>
+    </xacro:if>
   </xacro:macro>
+  <xacro:arg name="namespace" default="realsense" />
+  <xacro:arg name="parent" default="" />
+  <xacro:rcdt_zed2i namespace="$(arg namespace)" parent="$(arg parent)" />
 </robot>
