Commit message: WIP
Signed-off-by: Max Waterhout <max.waterhout@hotmail.nl>

File: ros2_ws/src/rcdt_sensors/urdf/rcdt_nmea_navsat.urdf.xacro (robot description, xacro)
@@ -7,12 +7,20 @@
 copied from:  https://github.com/husarion/husarion_components_description/blob/ros2/urdf/teltonika_003R-00253.urdf.xacro
 -->
-<robot xmlns:xacro="http://wiki.ros.org/xacro">
+<robot xmlns:xacro="http://wiki.ros.org/xacro" name="nmea_navsat">
   <xacro:macro name="teltonika_003R-00253"
-               params="parent_link
+               params="parent_link:=base_link
                        xyz:='0.0 0.0 0.0'
                        rpy:='0.0 0.0 0.0'
-                       namespace:=''
+                       namespace:=navsat
                        device_namespace:=gps">
     <xacro:property name="ns" value="${namespace + '/' if namespace != '' else ''}" />
+    <link name="base_link">
+      <inertial>
+        <origin xyz="0 0 0" rpy="0 0 0"/>
+        <mass value="0.001"/>
+        <inertia ixx="1e-6" iyy="1e-6" izz="1e-6"
+                ixy="0" ixz="0" iyz="0"/>
+      </inertial>
+    </link>
     <joint name="${parent_link.rstrip('_link')}_to_antenna_joint"
       type="fixed">
@@ -61,3 +69,9 @@
     </gazebo>
   </xacro:macro>
+  <xacro:teltonika_003R-00253
+      parent_link="base_link"
+      xyz="0.0 -0.06 0.55"
+      rpy="0.0 0.0 0.0"
+      namespace="navsat"
+      device_namespace="gps"/>
 </robot>

Commit message: Fix gps in simulation.
Signed-off-by: Jelmer de Wolde <jelmer.de.wolde@alliander.com>

File: ros2_ws/src/rcdt_sensors/urdf/rcdt_nmea_navsat.urdf.xacro (robot description, xacro)
@@ -4,66 +4,31 @@
 SPDX-License-Identifier: Apache-2.0
 -->
-<!--
-copied from:  https://github.com/husarion/husarion_components_description/blob/ros2/urdf/teltonika_003R-00253.urdf.xacro
--->
 <robot xmlns:xacro="http://wiki.ros.org/xacro" name="nmea_navsat">
-  <xacro:macro name="teltonika_003R-00253"
-               params="parent_link:=base_link
-                       xyz:='0.0 0.0 0.0'
-                       rpy:='0.0 0.0 0.0'
-                       namespace:=navsat
-                       device_namespace:=gps">
-    <xacro:property name="ns" value="${namespace + '/' if namespace != '' else ''}" />
-    <joint name="${parent_link.rstrip('_link')}_to_antenna_joint"
-      type="fixed">
-      <origin xyz="${xyz}" rpy="${rpy}" />
-      <parent link="${parent_link}" />
-      <child link="${device_namespace}_mounting_point" />
-    </joint>
-    <link name="${device_namespace}_mounting_point">
-      <visual>
-        <origin xyz="0.0 0.0 0.0" rpy="0.0 0.0 0.0" />
-        <geometry>
-          <mesh filename="package://husarion_components_description/meshes/teltonika_003R-00253.dae" />
-        </geometry>
-      </visual>
-      <collision>
-        <origin xyz="0.0 0.0 0.0" rpy="0.0 0.0 0.0" />
-        <geometry>
-          <mesh
-            filename="package://husarion_components_description/meshes/teltonika_003R-00253_collision.stl" />
-        </geometry>
-      </collision>
-      <inertial>
-        <origin xyz="0.045 0.0 0.0058" rpy="0.0 0.0 0.0" />
-        <mass value="0.59" />
-        <inertia ixx="0.003964" ixy="0.0000000" ixz="0.0"
-                                iyy="0.0003964" iyz="0.0"
-                                                izz="0.0004177" />
-      </inertial>
-    </link>
-    <joint
-      name="antenna_to_${device_namespace.rstrip('_link')}_joint"
-      type="fixed">
-      <origin xyz="0.045 0.0 0.0058" rpy="0.0 0.0 0.0" />
-      <parent link="${device_namespace}_mounting_point" />
-      <child link="${device_namespace}" />
-    </joint>
-    <link name="${device_namespace}" />
-    <gazebo reference="${device_namespace}">
-      <sensor name="navsat" type="navsat">
-        <plugin filename="ignition-gazebo-navsat-system" name="ignition::gazebo::systems::NavSat" />
-        <always_on>1</always_on>
-        <update_rate>1</update_rate>
-        <topic>${ns}${device_namespace}/fix</topic>
-        <gz_frame_id>${ns}${device_namespace}</gz_frame_id>
-      </sensor>
-    </gazebo>
-  </xacro:macro>
-  <xacro:teltonika_003R-00253
-      parent_link="base_link"
-      xyz="0.0 -0.06 0.55"
-      rpy="0.0 0.0 0.0"
-      namespace=""
-      device_namespace="gps"/>
+  <!-- Define arguments and related properties: -->
+  <xacro:arg name="namespace" default="" />
+  <xacro:arg name="parent" default="" />
+  <xacro:property name="namespace" value="$(arg namespace)" />
+  <xacro:property name="parent" value="$(arg parent)" />
+  <!-- Gazebo requires a joint to a link called "world" for statically mounted robots: -->
+  <xacro:if value="${parent != ''}">
+    <xacro:if value="${parent == 'world'}">
+      <link name="${parent}" />
+      <joint name="${parent}_joint" type="fixed">
+        <parent link="${parent}" />
+        <child link="base_link" />
+      </joint>
+    </xacro:if>
+  </xacro:if>
+  <!-- Gazebo requires a base link with inertia: -->
+  <link name="base_link">
+    <inertial>
+      <mass value="1e-10" />
+      <origin xyz="0 0 0" />
+      <inertia ixx="1" ixy="0" ixz="0" iyy="1" iyz="0" izz="1" />
+    </inertial>
+  </link>
+  <!-- Include teltonika xacro: -->
+  <xacro:include
+    filename="$(find husarion_components_description)/urdf/teltonika_003R-00253.urdf.xacro" />
+  <xacro:teltonika_003R-00253 parent_link="base_link" namespace="${namespace}" />
 </robot>
