Commit message: Remove unnecessary if statement.
Signed-off-by: Jelmer de Wolde <jelmer.de.wolde@alliander.com>

File: ros2_ws/src/rcdt_sensors/urdf/rcdt_axis.urdf.xacro (robot description, xacro)
@@ -12,12 +12,10 @@
     ">
     <!-- Gazebo requires a joint to a link called "world" for statically mounted robots -->
-    <xacro:if value="${parent != ''}">
-      <xacro:if value="${parent == 'world'}">
-        <link name="${parent}" />
-        <joint name="${parent}_joint" type="fixed">
-          <parent link="${parent}" />
-          <child link="base_link" />
-        </joint>
-      </xacro:if>
+    <xacro:if value="${parent == 'world'}">
+      <link name="${parent}" />
+      <joint name="${parent}_joint" type="fixed">
+        <parent link="${parent}" />
+        <child link="base_link" />
+      </joint>
     </xacro:if>
     <!-- Include realsense xacro: -->

File: ros2_ws/src/rcdt_sensors/urdf/rcdt_nmea_navsat.urdf.xacro (robot description, xacro)
@@ -11,12 +11,10 @@
   <xacro:property name="parent" value="$(arg parent)" />
   <!-- Gazebo requires a joint to a link called "world" for statically mounted robots: -->
-  <xacro:if value="${parent != ''}">
-    <xacro:if value="${parent == 'world'}">
-      <link name="${parent}" />
-      <joint name="${parent}_joint" type="fixed">
-        <parent link="${parent}" />
-        <child link="base_link" />
-      </joint>
-    </xacro:if>
+  <xacro:if value="${parent == 'world'}">
+    <link name="${parent}" />
+    <joint name="${parent}_joint" type="fixed">
+      <parent link="${parent}" />
+      <child link="base_link" />
+    </joint>
   </xacro:if>
   <!-- Gazebo requires a base link with inertia: -->

File: ros2_ws/src/rcdt_sensors/urdf/rcdt_realsense_d435.urdf.xacro (robot description, xacro)
@@ -14,12 +14,10 @@
     ">
     <!-- Gazebo requires a joint to a link called "world" for statically mounted robots -->
-    <xacro:if value="${parent != ''}">
-      <xacro:if value="${parent == 'world'}">
-        <link name="${parent}" />
-        <joint name="${parent}_joint" type="fixed">
-          <parent link="${parent}" />
-          <child link="base_link" />
-        </joint>
-      </xacro:if>
+    <xacro:if value="${parent == 'world'}">
+      <link name="${parent}" />
+      <joint name="${parent}_joint" type="fixed">
+        <parent link="${parent}" />
+        <child link="base_link" />
+      </joint>
     </xacro:if>
     <!-- Include realsense xacro: -->
@@ -78,4 +76,4 @@
   <xacro:arg name="namespace" default="realsense" />
   <xacro:arg name="parent" default="" />
-  <xacro:rcdt_realsense_d435 namespace="$(arg namespace)" parent="$(arg parent)"/>
+  <xacro:rcdt_realsense_d435 namespace="$(arg namespace)" parent="$(arg parent)" />
 </robot>

File: ros2_ws/src/rcdt_sensors/urdf/rcdt_velodyne.urdf.xacro (robot description, xacro)
@@ -69,12 +69,10 @@
     </link>
     <!-- Gazebo requires a joint to a link called "world" for statically mounted robots -->
-    <xacro:if value="${parent != ''}">
-      <xacro:if value="${parent == 'world'}">
-        <link name="${parent}" />
-        <joint name="${parent}_joint" type="fixed">
-          <parent link="${parent}" />
-          <child link="base_link" />
-        </joint>
-      </xacro:if>
+    <xacro:if value="${parent == 'world'}">
+      <link name="${parent}" />
+      <joint name="${parent}_joint" type="fixed">
+        <parent link="${parent}" />
+        <child link="base_link" />
+      </joint>
     </xacro:if>
     <gazebo reference="${name}">

File: ros2_ws/src/rcdt_sensors/urdf/rcdt_zed2i.urdf.xacro (robot description, xacro)
@@ -18,12 +18,10 @@
     ">
     <!-- Gazebo requires a joint to a link called "world" for statically mounted robots -->
-    <xacro:if value="${parent != ''}">
-      <xacro:if value="${parent == 'world'}">
-        <link name="${parent}" />
-        <joint name="${parent}_joint" type="fixed">
-          <parent link="${parent}" />
-          <child link="base_link" />
-        </joint>
-      </xacro:if>
+    <xacro:if value="${parent == 'world'}">
+      <link name="${parent}" />
+      <joint name="${parent}_joint" type="fixed">
+        <parent link="${parent}" />
+        <child link="base_link" />
+      </joint>
     </xacro:if>
     <!-- Gazebo requires a base link with inertia: -->
