Commit message: Define velodyne as separate 'robot'.
Signed-off-by: Jelmer de Wolde <jelmer.de.wolde@alliander.com>

File: ros2_ws/src/rcdt_panther/urdf/adapted/gazebo.urdf.xacro (robot description, xacro)
@@ -56,4 +56,14 @@
           <child_model>franka</child_model>
           <child_link>fr3_link0</child_link>
+        </plugin>
+      </gazebo>
+    </xacro:if>
+    <xacro:if value="${connected_to == 'velodyne'}">
+      <gazebo>
+        <plugin filename="libignition-gazebo-detachable-joint-system.so"
+          name="ignition::gazebo::systems::DetachableJoint">
+          <parent_link>base_link</parent_link>
+          <child_model>VLP-16</child_model>
+          <child_link>base_link</child_link>
         </plugin>
       </gazebo>

File: ros2_ws/src/rcdt_panther/urdf/panther.urdf.xacro (robot description, xacro)
@@ -18,11 +18,3 @@
     namespace="panther"
     connected_to="$(arg connected_to)" />
-  <!-- Load Velodyne: -->
-  <xacro:arg name="load_velodyne" default="false" />
-  <xacro:if value="$(arg load_velodyne)">
-    <xacro:include filename="$(find rcdt_sensors)/urdf/rcdt_velodyne.urdf.xacro" />
-    <xacro:VLP-16 namespace="panther">
-      <origin xyz="0.18 0 0.03" rpy="0 0 0" />
-    </xacro:VLP-16>
-  </xacro:if>
 </robot>

File: ros2_ws/src/rcdt_sensors/urdf/rcdt_velodyne.urdf.xacro (robot description, xacro)
@@ -15,6 +15,4 @@
     *origin
     namespace
-    parent:=cover_link
-    name:=velodyne
     update_rate:=10
     lasers:=16
@@ -25,10 +23,5 @@
     max_angle:=${M_PI}
     ">
-    <joint name="${name}_base_mount_joint" type="fixed">
-      <xacro:insert_block name="origin" />
-      <parent link="${parent}" />
-      <child link="${name}_base_link" />
-    </joint>
-    <link name="${name}_base_link">
+    <link name="base_link">
       <inertial>
         <mass value="0.83" />
@@ -55,10 +48,10 @@
       </collision>
     </link>
-    <joint name="${name}_base_scan_joint" type="fixed">
+    <joint name="base_scan_joint" type="fixed">
       <origin xyz="0 0 0.0377" rpy="0 0 0" />
-      <parent link="${name}_base_link" />
-      <child link="${name}_lidar" />
+      <parent link="base_link" />
+      <child link="lidar" />
     </joint>
-    <link name="${name}_lidar">
+    <link name="lidar">
       <inertial>
         <mass value="0.01" />
@@ -73,12 +66,12 @@
       </visual>
     </link>
-    <gazebo reference="${name}_lidar">
-      <sensor type="gpu_lidar" name="${name}">
+    <gazebo reference="lidar">
+      <sensor type="gpu_lidar" name="${namespace}">
         <always_on>true</always_on>
         <update_rate>${update_rate}</update_rate>
-        <topic>${namespace}/${name}/scan</topic>
+        <topic>${namespace}/scan</topic>
         <visualize>false</visualize>
-        <ignition_frame_id>${namespace}/${name}_lidar</ignition_frame_id>
-        <frame_id>${namespace}/${name}_lidar</frame_id>
+        <ignition_frame_id>${namespace}/lidar</ignition_frame_id>
+        <frame_id>${namespace}/lidar</frame_id>
         <ray>
           <scan>
@@ -110,3 +103,6 @@
     </gazebo>
   </xacro:macro>
+  <xacro:VLP-16 namespace="velodyne">
+    <origin xyz="0 0 0" rpy="0 0 0" />
+  </xacro:VLP-16>
 </robot>

Commit message: WIP
Signed-off-by: Max Waterhout <max.waterhout@hotmail.nl>

File: ros2_ws/src/rcdt_panther/urdf/adapted/gazebo.urdf.xacro (robot description, xacro)
@@ -2,5 +2,5 @@
 <!--
 Based on:
-https://github.com/husarion/husarion_ugv_ros/blob/2.1.2/panther_description/urdf/gazebo.urdf.xacro
+https://github.com/husarion/husarion_ugv_ros/blob/2.2.2/husarion_ugv_description/urdf/common/gazebo.urdf.xacro
 A copy of the original file is located in the /original directory.
 To compare the two files in VSCode, see:
@@ -37,5 +37,5 @@
   <xacro:macro name="controller" params="config_file namespace:=''">
     <gazebo>
-      <plugin filename="ign_ros2_control-system" name="ign_ros2_control::IgnitionROS2ControlPlugin">
+      <plugin filename="gz_ros2_control-system" name="gz_ros2_control::GazeboSimROS2ControlPlugin">
         <parameters>${config_file}</parameters>
         <ros>
@@ -117,5 +117,5 @@
   <xacro:macro name="light" params="reference_frame name topic namespace:=''">
     <gazebo>
-      <plugin filename="LEDStrip" name="panther_gazebo::LEDStrip">
+      <plugin filename="LEDStrip" name="husarion_ugv_gazebo::LEDStrip">
         <light_name>${name}</light_name>
         <topic>${topic}</topic>

File: ros2_ws/src/rcdt_panther/urdf/adapted/panther_macro.urdf.xacro (robot description, xacro)
@@ -10,6 +10,5 @@
   <xacro:macro
     name="panther_robot"
-    params="panther_version
-            wheel_config_file
+    params="wheel_config_file
             controller_config_file
             battery_config_file
@@ -19,6 +18,4 @@
             namespace:=''
             connected_to:=''">
-    <!-- Map params to args: -->
-    <xacro:arg name="use_sim" default="${use_sim}" />
     <xacro:if value="${use_sim}">
       <xacro:property name="imu_xyz" value="-0.195 0.010 0.085" />
@@ -27,9 +24,10 @@
     <xacro:property name="ns" value='${namespace + "/" if namespace else ""}' />
     <xacro:property name="wheel_config" value="${xacro.load_yaml(wheel_config_file)}" />
-    <xacro:property name="wheel_separation_x" value="0.44" />
+    <xacro:property name="wheelbase" value="0.44" />
+    <xacro:property name="wheel_mount_point_y" value="0.2575" />
     <!-- INCLUDE ROBOT PARTS DEFINITIONS -->
-    <xacro:include filename="$(find panther_description)/urdf/body.urdf.xacro" ns="body" />
+    <xacro:include filename="$(find husarion_ugv_description)/urdf/panther/base.urdf.xacro" ns="body" />
     <xacro:include filename="$(find rcdt_panther)/urdf/adapted/gazebo.urdf.xacro" ns="gazebo" />
-    <xacro:include filename="$(find panther_description)/urdf/wheel.urdf.xacro" ns="wheel" />
+    <xacro:include filename="$(find husarion_ugv_description)/urdf/common/wheel.urdf.xacro" ns="wheel" />
     <!-- BODY DECLARATION -->
     <xacro:body.body
@@ -39,28 +37,31 @@
     <!-- WHEEL DECLARATION -->
     <xacro:wheel.wheel
-      wheel_config="${wheel_config}"
-      wheel_separation_x="${wheel_separation_x}"
+      config="${wheel_config}"
+      mount_point_x="${wheelbase/2.0}"
+      mount_point_y="${wheel_mount_point_y}"
       prefix="fl" />
     <xacro:wheel.wheel
-      wheel_config="${wheel_config}"
-      wheel_separation_x="${wheel_separation_x}"
+      config="${wheel_config}"
+      mount_point_x="${wheelbase/2.0}"
+      mount_point_y="${wheel_mount_point_y}"
       prefix="fr" />
     <xacro:wheel.wheel
-      wheel_config="${wheel_config}"
-      wheel_separation_x="${wheel_separation_x}"
+      config="${wheel_config}"
+      mount_point_x="${wheelbase/2.0}"
+      mount_point_y="${wheel_mount_point_y}"
       prefix="rl" />
     <xacro:wheel.wheel
-      wheel_config="${wheel_config}"
-      wheel_separation_x="${wheel_separation_x}"
+      config="${wheel_config}"
+      mount_point_x="${wheelbase/2.0}"
+      mount_point_y="${wheel_mount_point_y}"
       prefix="rr" />
     <ros2_control name="${ns}panther_system" type="system">
       <hardware>
         <xacro:if value="${use_sim}">
-          <plugin>panther_gazebo/GzPantherSystem</plugin>
+          <plugin>husarion_ugv_gazebo/EStopSystem</plugin>
           <param name="e_stop_initial_state">true</param>
         </xacro:if>
-        <xacro:unless value="$(arg use_sim)">
-          <plugin>panther_hardware_interfaces/PantherSystem</plugin>
-          <param name="panther_version">${panther_version}</param>
+        <xacro:unless value="${use_sim}">
+          <plugin>husarion_ugv_hardware_interfaces/PantherSystem</plugin>
           <param name="encoder_resolution">1600</param>
           <param name="gear_ratio">30.08</param>
@@ -70,5 +71,5 @@
           <!-- Max RPM speed set in the Roboteq driver (MXRPM parameter) -->
           <param name="max_rpm_motor_speed">3600.0</param>
-          <param name="can_interface_name">panther_can</param>
+          <param name="can_interface_name">robot_can</param>
           <param name="master_can_id">3</param>
           <param name="front_driver_can_id">1</param>
@@ -129,8 +130,8 @@
       </xacro:if>
     </ros2_control>
-    <xacro:unless value="$(arg use_sim)">
+    <xacro:unless value="${use_sim}">
       <ros2_control name="${ns}imu" type="sensor">
         <hardware>
-          <plugin>panther_hardware_interfaces/PantherImuSensor</plugin>
+          <plugin>husarion_ugv_hardware_interfaces/PhidgetImuSensor</plugin>
           <param name="serial">-1</param>
           <param name="hub_port">0</param>

File: ros2_ws/src/rcdt_panther/urdf/panther.urdf.xacro (robot description, xacro)
@@ -11,7 +11,6 @@
   <xacro:include filename="$(find rcdt_panther)/urdf/adapted/panther_macro.urdf.xacro" ns="husarion" />
   <xacro:husarion.panther_robot
-    panther_version="1.0"
     use_sim="$(arg simulation)"
-    wheel_config_file="$(find panther_description)/config/WH01.yaml"
+    wheel_config_file="$(find husarion_ugv_description)/config/WH01.yaml"
     controller_config_file="$(find rcdt_gazebo)/config/controllers.yaml"
     battery_config_file=""

Commit message: Add nav2 to the panther (#198)
* Update environment variables for the meshes

Signed-off-by: Max Waterhout <max.waterhout@hotmail.nl>

* Enable nav2 navigation to panther.launch

Signed-off-by: Max Waterhout <max.waterhout@hotmail.nl>

* Add nav2 launch file and integration tests for Panther navigation

Signed-off-by: Max Waterhout <max.waterhout@hotmail.nl>

* Remove redundant navigation launch instructions from Panther documentation

Signed-off-by: Max Waterhout <max.waterhout@hotmail.nl>

* Refactor navigation launch setup: replace navigation.launch.py with nav2.launch.py and update launch arguments

Signed-off-by: Max Waterhout <max.waterhout@hotmail.nl>

* Add collision monitor argument to navigation launch files

Signed-off-by: Max Waterhout <max.waterhout@hotmail.nl>

* Update build cache reference in reusable-docker.yml to use 'build-cache-latest'

Signed-off-by: Max Waterhout <max.waterhout@hotmail.nl>

* Update test_panther_nav2.py: Enable RViz and adjust navigation goal position and orientation

Signed-off-by: Max Waterhout <max.waterhout@hotmail.nl>

* Refactor test_panther_nav2.py: Disable RViz and remove unnecessary sleep in registration test

Signed-off-by: Max Waterhout <max.waterhout@hotmail.nl>

* Add support for real lidar.

Signed-off-by: Jelmer de Wolde <jelmer.de.wolde@alliander.com>

* Define velodyne as separate 'robot'.

Signed-off-by: Jelmer de Wolde <jelmer.de.wolde@alliander.com>

* Fix reuse.

Signed-off-by: Jelmer de Wolde <jelmer.de.wolde@alliander.com>

* Add velodyne packages to docker image.

Signed-off-by: Jelmer de Wolde <jelmer.de.wolde@alliander.com>

* Fix parameters.

Signed-off-by: Jelmer de Wolde <jelmer.de.wolde@alliander.com>

* Fix spawn position of panther.

Signed-off-by: Jelmer de Wolde <jelmer.de.wolde@alliander.com>

* Set nav2 default to false.

Signed-off-by: Jelmer de Wolde <jelmer.de.wolde@alliander.com>

* Remove old panther namespace.

Signed-off-by: Jelmer de Wolde <jelmer.de.wolde@alliander.com>

* Enable nav2 in launch file for test.

Signed-off-by: Jelmer de Wolde <jelmer.de.wolde@alliander.com>

* Fix for use on real robot.

Signed-off-by: Jelmer de Wolde <jelmer.de.wolde@alliander.com>

* Update transform_tolerance in controller_server parameters to improve navigation stability

Signed-off-by: Max Waterhout <max.waterhout@hotmail.nl>

* Add velodyne robot model to rviz.

Signed-off-by: Jelmer de Wolde <jelmer.de.wolde@alliander.com>

---------

Signed-off-by: Max Waterhout <max.waterhout@hotmail.nl>
Signed-off-by: Jelmer de Wolde <jelmer.de.wolde@alliander.com>

File: ros2_ws/src/rcdt_panther/urdf/adapted/gazebo.urdf.xacro (robot description, xacro)
@@ -54,4 +54,14 @@
           <child_model>franka</child_model>
           <child_link>fr3_link0</child_link>
+        </plugin>
+      </gazebo>
+    </xacro:if>
+    <xacro:if value="${connected_to == 'velodyne'}">
+      <gazebo>
+        <plugin filename="libignition-gazebo-detachable-joint-system.so"
+          name="ignition::gazebo::systems::DetachableJoint">
+          <parent_link>base_link</parent_link>
+          <child_model>VLP-16</child_model>
+          <child_link>base_link</child_link>
         </plugin>
       </gazebo>

File: ros2_ws/src/rcdt_panther/urdf/panther.urdf.xacro (robot description, xacro)
@@ -18,11 +18,3 @@
     namespace="panther"
     connected_to="$(arg connected_to)" />
-  <!-- Load Velodyne: -->
-  <xacro:arg name="load_velodyne" default="false" />
-  <xacro:if value="$(arg load_velodyne)">
-    <xacro:include filename="$(find rcdt_sensors)/urdf/rcdt_velodyne.urdf.xacro" />
-    <xacro:VLP-16 namespace="panther">
-      <origin xyz="0.18 0 0.03" rpy="0 0 0" />
-    </xacro:VLP-16>
-  </xacro:if>
 </robot>

File: ros2_ws/src/rcdt_sensors/urdf/rcdt_velodyne.urdf.xacro (robot description, xacro)
@@ -7,5 +7,5 @@
 Based on:
 1.https://bitbucket.org/DataspeedInc/velodyne_simulator/src/master/velodyne_description/urdf/VLP-16.urdf.xacro
-2.https://github.com/husarion/ros_components_description/blob/ros2/urdf/velodyne_puck.urdf.xacro
+2.https://github.com/husarion/husarion_components_description/blob/ros2/urdf/velodyne_puck.urdf.xacro
 -->
 <robot xmlns:xacro="http://www.ros.org/wiki/xacro" name="VLP-16">
@@ -15,5 +15,4 @@
     *origin
     namespace
-    parent:=cover_link
     name:=velodyne
     update_rate:=10
@@ -25,10 +24,5 @@
     max_angle:=${M_PI}
     ">
-    <joint name="${name}_base_mount_joint" type="fixed">
-      <xacro:insert_block name="origin" />
-      <parent link="${parent}" />
-      <child link="${name}_base_link" />
-    </joint>
-    <link name="${name}_base_link">
+    <link name="base_link">
       <inertial>
         <mass value="0.83" />
@@ -55,10 +49,10 @@
       </collision>
     </link>
-    <joint name="${name}_base_scan_joint" type="fixed">
+    <joint name="base_scan_joint" type="fixed">
       <origin xyz="0 0 0.0377" rpy="0 0 0" />
-      <parent link="${name}_base_link" />
-      <child link="${name}_lidar" />
+      <parent link="base_link" />
+      <child link="${name}" />
     </joint>
-    <link name="${name}_lidar">
+    <link name="${name}">
       <inertial>
         <mass value="0.01" />
@@ -73,12 +67,12 @@
       </visual>
     </link>
-    <gazebo reference="${name}_lidar">
-      <sensor type="gpu_lidar" name="${name}">
+    <gazebo reference="${name}">
+      <sensor type="gpu_lidar" name="${namespace}">
         <always_on>true</always_on>
         <update_rate>${update_rate}</update_rate>
-        <topic>${namespace}/${name}/scan</topic>
+        <topic>${namespace}/scan</topic>
         <visualize>false</visualize>
-        <gz_frame_id>${namespace}/${name}_lidar</gz_frame_id>
-        <frame_id>${namespace}/${name}_lidar</frame_id>
+        <gz_frame_id>${namespace}/${name}</gz_frame_id>
+        <frame_id>${namespace}/${name}</frame_id>
         <ray>
           <scan>
@@ -110,3 +104,6 @@
     </gazebo>
   </xacro:macro>
+  <xacro:VLP-16 namespace="velodyne">
+    <origin xyz="0 0 0" rpy="0 0 0" />
+  </xacro:VLP-16>
 </robot>

Commit message: WIP
Signed-off-by: Jelmer de Wolde <jelmer.de.wolde@alliander.com>

File: ros2_ws/src/rcdt_panther/urdf/adapted/gazebo.urdf.xacro (robot description, xacro)
@@ -45,27 +45,4 @@
     </gazebo>
   </xacro:macro>
-  <!-- Detachable joint: -->
-  <xacro:macro name="detachable_joint" params="connected_to:=''">
-    <xacro:if value="${connected_to == 'franka'}">
-      <gazebo>
-        <plugin filename="gz-sim-detachable-joint-system"
-          name="gz::sim::systems::DetachableJoint">
-          <parent_link>base_link</parent_link>
-          <child_model>franka</child_model>
-          <child_link>fr3_link0</child_link>
-        </plugin>
-      </gazebo>
-    </xacro:if>
-    <xacro:if value="${connected_to == 'velodyne'}">
-      <gazebo>
-        <plugin filename="libignition-gazebo-detachable-joint-system.so"
-          name="ignition::gazebo::systems::DetachableJoint">
-          <parent_link>base_link</parent_link>
-          <child_model>VLP-16</child_model>
-          <child_link>base_link</child_link>
-        </plugin>
-      </gazebo>
-    </xacro:if>
-  </xacro:macro>
   <!-- Gauss noise macro -->
   <xacro:macro name="gauss_noise"
@@ -79,6 +56,5 @@
     </noise>
   </xacro:macro>
-  <!-- IMU specification:
-  https://www.phidgets.com/?tier=3&catid=10&pcid=8&prodid=1025#Tab_Specifications -->
+  <!-- IMU specification: https://www.phidgets.com/?tier=3&catid=10&pcid=8&prodid=1025#Tab_Specifications -->
   <xacro:macro name="imu" params="reference_frame namespace:=''">
     <xacro:property name="ns" value='${namespace + "/" if namespace else ""}' />
@@ -90,5 +66,5 @@
         <visualize>false</visualize>
         <enable_metrics>false</enable_metrics>
-        <!-- <gz_frame_id>imu_link</gz_frame_id> -->
+        <gz_frame_id>imu_link</gz_frame_id>
         <imu>
           <orientation_reference_frame>

File: ros2_ws/src/rcdt_panther/urdf/adapted/panther_macro.urdf.xacro (robot description, xacro)
@@ -16,6 +16,5 @@
             imu_xyz:='0.169 0.025 0.092'
             imu_rpy:='0.0 0.0 -1.57'
-            namespace:=''
-            connected_to:=''">
+            namespace:=''">
     <xacro:if value="${use_sim}">
       <xacro:property name="imu_xyz" value="-0.195 0.010 0.085" />
@@ -168,5 +167,4 @@
       </xacro:if>
       <xacro:gazebo.controller config_file="${controller_config_file}" namespace="${namespace}" />
-      <xacro:gazebo.detachable_joint connected_to="${connected_to}"/>
       <xacro:gazebo.imu reference_frame="imu_link" namespace="${namespace}" />
       <xacro:gazebo.light reference_frame="lights_channel_1_link" name="lights_channel_1" topic="lights/channel_1_frame" namespace="${namespace}" />

File: ros2_ws/src/rcdt_panther/urdf/panther.urdf.xacro (robot description, xacro)
@@ -7,5 +7,6 @@
   <!-- Set use_sim argument to let panther xacro load gazebo plugin: -->
   <xacro:arg name="simulation" default="true" />
-  <xacro:arg name="connected_to" default="" />
+  <xacro:arg name="namespace" default="panther" />
+  <xacro:arg name="childs" default="${[]}" />
   <!-- Load panther: -->
   <xacro:include filename="$(find rcdt_panther)/urdf/adapted/panther_macro.urdf.xacro"
@@ -16,5 +17,7 @@
     controller_config_file="$(find rcdt_gazebo)/config/controllers.yaml"
     battery_config_file=""
-    namespace="panther"
-    connected_to="$(arg connected_to)" />
+    namespace="$(arg namespace)" />
+  <!-- Create detachable joints between base_link and childs: -->
+  <xacro:include filename="$(find rcdt_utilities)/urdf/detachable_joints.urdf.xacro" />
+  <xacro:detachable_joints parent_link="base_link" childs="${$(arg childs)}" />
 </robot>

Commit message: Add moving block control node and update world configurations for simulation
Signed-off-by: Max Waterhout <max.waterhout@hotmail.nl>

File: ros2_ws/src/rcdt_panther/urdf/adapted/gazebo.urdf.xacro (robot description, xacro)
@@ -42,4 +42,13 @@
           <namespace>${namespace}</namespace>
         </ros>
+      </plugin>
+    </gazebo>
+  </xacro:macro>
+  <xacro:macro name="odom_publisher">
+    <gazebo>
+        <plugin
+        filename="gz-sim-odometry-publisher-system"
+        name="gz::sim::systems::OdometryPublisher">
+        <dimensions>3</dimensions>
       </plugin>
     </gazebo>

File: ros2_ws/src/rcdt_panther/urdf/adapted/panther_macro.urdf.xacro (robot description, xacro)
@@ -168,4 +168,5 @@
       </xacro:if>
       <xacro:gazebo.controller config_file="${controller_config_file}" namespace="${namespace}" />
+      <xacro:gazebo.odom_publisher />
       <xacro:gazebo.detachable_joint connected_to="${connected_to}"/>
       <xacro:gazebo.imu reference_frame="imu_link" namespace="${namespace}" />

Commit message: WIP
Signed-off-by: Max Waterhout <max.waterhout@hotmail.nl>

File: ros2_ws/src/rcdt_panther/urdf/adapted/gazebo.urdf.xacro (robot description, xacro)
@@ -44,4 +44,37 @@
       </plugin>
     </gazebo>
+  </xacro:macro>
+  <!-- Detachable joint: -->
+  <xacro:macro name="detachable_joint" params="connected_to:=''">
+    <xacro:if value="${connected_to == 'franka'}">
+      <gazebo>
+        <plugin filename="gz-sim-detachable-joint-system"
+          name="gz::sim::systems::DetachableJoint">
+          <parent_link>base_link</parent_link>
+          <child_model>franka</child_model>
+          <child_link>fr3_link0</child_link>
+        </plugin>
+      </gazebo>
+    </xacro:if>
+    <xacro:if value="${connected_to == 'velodyne'}">
+      <gazebo>
+        <plugin filename="libignition-gazebo-detachable-joint-system.so"
+          name="ignition::gazebo::systems::DetachableJoint">
+          <parent_link>base_link</parent_link>
+          <child_model>VLP-16</child_model>
+          <child_link>base_link</child_link>
+        </plugin>
+      </gazebo>
+    </xacro:if>
+    <xacro:if value="${connected_to == 'navsat'}">
+      <gazebo>
+        <plugin filename="libignition-gazebo-detachable-joint-system.so"
+          name="ignition::gazebo::systems::DetachableJoint">
+          <parent_link>base_link</parent_link>
+          <child_model>nmea_navsat</child_model>
+          <child_link>gps_mounting_point</child_link>
+        </plugin>
+      </gazebo>
+    </xacro:if>
   </xacro:macro>
   <!-- Gauss noise macro -->

File: ros2_ws/src/rcdt_sensors/urdf/rcdt_nmea_navsat.urdf.xacro (robot description, xacro)
@@ -15,12 +15,4 @@
                        device_namespace:=gps">
     <xacro:property name="ns" value="${namespace + '/' if namespace != '' else ''}" />
-    <link name="base_link">
-      <inertial>
-        <origin xyz="0 0 0" rpy="0 0 0"/>
-        <mass value="0.001"/>
-        <inertia ixx="1e-6" iyy="1e-6" izz="1e-6"
-                ixy="0" ixz="0" iyz="0"/>
-      </inertial>
-    </link>
     <joint name="${parent_link.rstrip('_link')}_to_antenna_joint"
       type="fixed">
@@ -73,5 +65,5 @@
       xyz="0.0 -0.06 0.55"
       rpy="0.0 0.0 0.0"
-      namespace="navsat"
+      namespace=""
       device_namespace="gps"/>
 </robot>
