Commit message: Move camera for better view.
Signed-off-by: Jelmer de Wolde <jelmer.de.wolde@alliander.com>

File: ros2_ws/src/rcdt_franka/urdf/franka.urdf.xacro (robot description, xacro)
@@ -41,5 +41,5 @@
     <link name="realsense_link" />
     <joint name="realsense_link_joint" type="fixed">
-      <origin xyz="0.02 0 0.05" rpy="0 ${-0.5*pi} ${pi}" />
+      <origin xyz="0.05 0 0.05" rpy="0 ${-0.5*pi} ${pi}" />
       <parent link="fr3_hand" />
       <child link="realsense_link" />

Commit message: Changes for test on real robot.
Signed-off-by: Jelmer de Wolde <jelmer.de.wolde@alliander.com>

File: ros2_ws/src/rcdt_franka/urdf/franka.urdf.xacro (robot description, xacro)
@@ -41,5 +41,5 @@
     <link name="realsense_link" />
     <joint name="realsense_link_joint" type="fixed">
-      <origin xyz="0.05 0 0.05" rpy="0 ${-0.5*pi} ${pi}" />
+      <origin xyz="0.05 0 0.01" rpy="0 ${-0.5*pi} ${pi}" />
       <parent link="fr3_hand" />
       <child link="realsense_link" />

Commit message: Improve camera position.
Signed-off-by: Jelmer de Wolde <jelmer.de.wolde@alliander.com>

File: ros2_ws/src/rcdt_franka/urdf/franka.urdf.xacro (robot description, xacro)
@@ -41,5 +41,5 @@
     <link name="realsense_link" />
     <joint name="realsense_link_joint" type="fixed">
-      <origin xyz="0.05 0 0.01" rpy="0 ${-0.5*pi} ${pi}" />
+      <origin xyz="0.05 -0.02 0.01" rpy="0 ${-0.5*pi} ${pi}" />
       <parent link="fr3_hand" />
       <child link="realsense_link" />

Commit message: finetuning
Signed-off-by: Yuri van Warmerdam <yuri.van.warmerdam@alliander.com>

File: ros2_ws/src/rcdt_franka/urdf/franka.urdf.xacro (robot description, xacro)
@@ -41,5 +41,5 @@
     <link name="realsense_link" />
     <joint name="realsense_link_joint" type="fixed">
-      <origin xyz="0.05 -0.02 0.01" rpy="0 ${-0.5*pi} ${pi}" />
+      <origin xyz="0.05 0 0.01" rpy="0 ${-0.5*pi} ${pi}" />
       <parent link="fr3_hand" />
       <child link="realsense_link" />

File: ros2_ws/src/rcdt_sensors/urdf/rcdt_realsense_d435.urdf.xacro (robot description, xacro)
@@ -21,5 +21,5 @@
       parent="${parent}"
       use_nominal_extrinsics="true">
-      <origin xyz="0 0 0" rpy="0 0 0" />
+      <origin xyz="0 0.015 0" rpy="0 0 0" />
     </xacro:sensor_d435>
     <!-- Add gazebo plugin: -->
@@ -28,4 +28,5 @@
         <!-- rgb_camera: -->
         <sensor type="camera" name="${namespace}_intel_realsense_d435_color">
+          <!-- <pose>0 -0.04 0 0 0 0</pose> -->
           <always_on>true</always_on>
           <update_rate>30.0</update_rate>
@@ -47,4 +48,5 @@
         <!-- depth camera -->
         <sensor type="depth_camera" name="${namespace}_intel_realsense_d435_depth">
+          <!-- <pose>0 -0.04 0 0 0 0</pose> -->
           <always_on>true</always_on>
           <update_rate>30.0</update_rate>

Commit message: Refactor robot cores.
Signed-off-by: Jelmer de Wolde <jelmer.de.wolde@alliander.com>

File: ros2_ws/src/rcdt_franka/urdf/franka.urdf.xacro (robot description, xacro)
@@ -5,36 +5,45 @@
 -->
 <robot xmlns:xacro="http://www.ros.org/wiki/xacro" name="franka">
-  <!-- Global Franka definitions: -->
+  <!-- arguments: -->
   <xacro:arg name="arm_id" default="fr3" />
   <xacro:arg name="ee_id" default="franka_hand" />
-  <!-- Franka related: -->
+  <xacro:arg name="namespace" default="" />
   <xacro:arg name="parent" default="world" />
   <xacro:arg name="xyz" default="0 0 0" />
   <xacro:arg name="gazebo" default="false" />
-  <xacro:arg name="ign_ros2_control" default="false" />
   <xacro:arg name="robot_ip" default="" />
-  <!-- Realsense related: -->
   <xacro:arg name="load_realsense" default="false" />
-  <!-- Load arm: -->
-  <xacro:include filename="$(find franka_description)/robots/common/franka_robot.xacro" />
+  <!-- robot definition: -->
+  <xacro:include filename="$(find rcdt_franka)/urdf/franka_robot.urdf.xacro" />
   <xacro:franka_robot
-    arm_id="$(arg arm_id)"
-    joint_limits="${xacro.load_yaml('$(find franka_description)/robots/$(arg arm_id)/joint_limits.yaml')}"
-    inertials="${xacro.load_yaml('$(find franka_description)/robots/$(arg arm_id)/inertials.yaml')}"
-    kinematics="${xacro.load_yaml('$(find franka_description)/robots/$(arg arm_id)/kinematics.yaml')}"
-    dynamics="${xacro.load_yaml('$(find franka_description)/robots/$(arg arm_id)/dynamics.yaml')}"
+    arm_id="fr3"
+    joint_limits="${xacro.load_yaml('$(find franka_description)/robots/fr3/joint_limits.yaml')}"
+    inertials="${xacro.load_yaml('$(find franka_description)/robots/fr3/inertials.yaml')}"
+    kinematics="${xacro.load_yaml('$(find franka_description)/robots/fr3/kinematics.yaml')}"
+    dynamics="${xacro.load_yaml('$(find franka_description)/robots/fr3/dynamics.yaml')}"
+    gazebo="$(arg gazebo)"
+    ee_id="$(arg ee_id)"
     parent="$(arg parent)"
-    ee_id="$(arg ee_id)"
-    gazebo="$(arg gazebo)"
-    xyz="$(arg xyz)" />
-  <!-- Load ros2 control. gazebo to LOAD and USE plugin. ign_ros2_control to only USE plugin. -->
-  <xacro:include filename="$(find franka_description)/robots/common/franka_arm.ros2_control.xacro" />
-  <xacro:franka_arm_ros2_control
+  />
+  <!-- ros2_control definition: -->
+  <xacro:include filename="$(find rcdt_franka)/urdf/franka_ros2_control.urdf.xacro" />
+  <xacro:franka_ros2_control
     arm_id="$(arg arm_id)"
     robot_ip="$(arg robot_ip)"
+    gazebo="$(arg gazebo)"
     hand="true"
-    gazebo="$(arg gazebo)"
-    ign_ros2_control="$(arg ign_ros2_control)" />
-  <!-- Load realsense: -->
+  />
+  <!-- gazebo plugins: -->
+  <gazebo>
+    <plugin filename="ign_ros2_control-system" name="ign_ros2_control::IgnitionROS2ControlPlugin">
+      <parameters>$(find rcdt_gazebo)/config/controllers.yaml</parameters>
+      <ros>
+        <namespace>$(arg namespace)</namespace>
+        <xacro:include filename="$(find rcdt_gazebo)/urdf/remappings.urdf.xacro" />
+        <xacro:remappings />
+      </ros>
+    </plugin>
+  </gazebo>
+  <!-- realsense: -->
   <xacro:if value="$(arg load_realsense)">
     <xacro:include filename="$(find rcdt_sensors)/urdf/rcdt_realsense_d435.urdf.xacro" />

File: ros2_ws/src/rcdt_panther/urdf/panther.urdf.xacro (robot description, xacro)
@@ -1,26 +1,44 @@
-<?xml version="1.0" encoding="utf-8"?>
+<?xml version='1.0' encoding='utf-8'?>
 <!--
 SPDX-FileCopyrightText: Alliander N. V.
 SPDX-License-Identifier: Apache-2.0
 -->
-<robot xmlns:xacro="http://wiki.ros.org/xacro" name="panther">
-  <!-- Set use_sim argument to let panther xacro load gazebo plugin: -->
-  <xacro:arg name="use_sim" default="true" />
-  <!-- Load panther: -->
-  <xacro:include filename="$(find panther_description)/urdf/panther_macro.urdf.xacro" ns="husarion" />
-  <xacro:husarion.panther_robot
+<robot xmlns:xacro="http://www.ros.org/wiki/xacro" name="panther">
+  <!-- arguments: -->
+  <xacro:arg name="namespace" default="" />
+  <xacro:arg name="connect_with_franka" default="false" />
+  <!-- robot definition: -->
+  <xacro:include filename="$(find rcdt_panther)/urdf/panther_robot.urdf.xacro" />
+  <xacro:panther_robot
     panther_version="1.0"
-    use_sim="$(arg use_sim)"
     wheel_config_file="$(find panther_description)/config/WH01.yaml"
-    controller_config_file="$(find rcdt_panther)/config/ros_controller.yaml"
-    battery_config_file=""
-    namespace="panther" />
-  <!-- Load Velodyne: -->
-  <xacro:arg name="load_velodyne" default="false" />
-  <xacro:if value="$(arg load_velodyne)">
-    <xacro:include filename="$(find rcdt_sensors)/urdf/rcdt_velodyne.urdf.xacro" />
-    <xacro:VLP-16 namespace="panther">
-      <origin xyz="0.18 0 0.03" rpy="0 0 0" />
-    </xacro:VLP-16>
-  </xacro:if>
+    namespace="$(arg namespace)"
+  />
+  <!-- ros2_control definition: -->
+  <xacro:include filename="$(find rcdt_panther)/urdf/panther_ros2_control.urdf.xacro" />
+  <xacro:panther_ros2_control
+    panther_version="1.0"
+    use_sim="true"
+    namespace="$(arg namespace)"
+  />
+  <!-- gazebo plugins: -->
+  <gazebo>
+    <plugin filename="ign_ros2_control-system" name="ign_ros2_control::IgnitionROS2ControlPlugin">
+      <parameters>$(find rcdt_gazebo)/config/controllers.yaml</parameters>
+      <ros>
+        <namespace>$(arg namespace)</namespace>
+        <xacro:include filename="$(find rcdt_gazebo)/urdf/remappings.urdf.xacro" />
+        <xacro:remappings />
+      </ros>
+    </plugin>
+    <xacro:if value="$(arg connect_with_franka)">
+      <plugin filename="libignition-gazebo-detachable-joint-system.so"
+        name="ignition::gazebo::systems::DetachableJoint">
+        <parent_link>base_link</parent_link>
+        <child_model>franka</child_model>
+        <child_link>link_to_panther</child_link>
+      </plugin>
+    </xacro:if>
+  </gazebo>
+  <!-- velodyne: -->
 </robot>

Commit message: Add ZED2i camera support in URDF and launch files
Signed-off-by: Max Waterhout <max.waterhout@hotmail.nl>

File: ros2_ws/src/rcdt_franka/urdf/franka.urdf.xacro (robot description, xacro)
@@ -10,4 +10,5 @@
   <xacro:arg name="parent" default="world" />
   <xacro:arg name="load_realsense" default="false" />
+  <xacro:arg name="load_zed2i"      default="true"/>   <!-- new -->
   <!-- robot: -->
   <xacro:include filename="$(find rcdt_franka)/urdf/adapted/franka_robot.xacro" />
@@ -41,3 +42,21 @@
     />
   </xacro:if>
+<xacro:include filename="$(find rcdt_sensors)/urdf/rcdt_zed2i.urdf.xacro" />
+<link  name="zed2i_link"/>
+<joint name="zed2i_link_joint" type="fixed">
+  <origin xyz="0.1 -0.02 0.01" rpy="0 0 0"/>
+  <parent link="fr3_hand"/>
+  <child  link="zed2i_link"/>
+</joint>
+<!-- Instantiate the camera subtree -->
+<xacro:rcdt_zed2i
+      robot_namespace="$(arg namespace)"
+      device_namespace="zed2i"
+      parent="zed2i_link"/>
+<joint name="zed2i_mount_joint" type="fixed">
+  <!-- pose of the camera w.r.t. the adapter; adjust if needed -->
+  <origin xyz="0 0 0" rpy="0 0 0"/>
+  <parent link="zed2i_link"/>
+  <child  link="zed2i_camera_link"/>   <!-- root link inside the macro -->
+</joint>
 </robot>

Commit message: WIP
Signed-off-by: Jelmer de Wolde <jelmer.de.wolde@alliander.com>

File: ros2_ws/src/rcdt_franka/urdf/franka.urdf.xacro (robot description, xacro)
@@ -16,4 +16,5 @@
   <xacro:arg name="parent" default="world" />
   <xacro:arg name="load_realsense" default="false" />
+  <xacro:arg name="childs" default="${[]}" />
   <!-- robot: -->
   <xacro:include filename="$(find rcdt_franka)/urdf/adapted/franka_robot.xacro" />
@@ -35,19 +36,6 @@
     parent="$(arg parent)"
   />
-  <!-- realsense: -->
-  <xacro:if value="$(arg load_realsense)">
-    <xacro:include filename="$(find rcdt_sensors)/urdf/rcdt_realsense_d435.urdf.xacro" />
-    <link name="realsense_link" />
-    <joint name="realsense_link_joint" type="fixed">
-      <origin xyz="0.05 -0.02 0.01" rpy="0 ${-0.5*pi} ${pi}" />
-      <parent link="fr3_hand" />
-      <child link="realsense_link" />
-    </joint>
-    <xacro:rcdt_realsense_d435
-      robot_namespace="$(arg namespace)"
-      device_namespace="realsense"
-      parent="realsense_link"
-      gazebo="$(arg simulation)"
-    />
-  </xacro:if>
+  <!-- Create detachable joints between base_link and childs: -->
+  <xacro:include filename="$(find rcdt_utilities)/urdf/detachable_joints.urdf.xacro" />
+  <xacro:detachable_joints parent_link="fr3_link0" childs="${$(arg childs)}" />
 </robot>

Commit message: 268 Create a modular launch system (#266)
Introduce a modular launch system.

---------

Signed-off-by: Jelmer de Wolde <jelmer.de.wolde@alliander.com>

File: ros2_ws/src/rcdt_franka/urdf/franka.urdf.xacro (robot description, xacro)
@@ -15,5 +15,6 @@
   <xacro:arg name="simulation" default="false" />
   <xacro:arg name="parent" default="world" />
-  <xacro:arg name="load_realsense" default="false" />
+  <xacro:arg name="childs" default="${[]}" />
+  <xacro:arg name="ip_address" default="" />
   <!-- robot: -->
   <xacro:include filename="$(find rcdt_franka)/urdf/adapted/franka_robot.xacro" />
@@ -31,23 +32,10 @@
     tcp_rpy="$(arg tcp_rpy)"
     ros2_control="true"
-    robot_ip="10.15.20.4"
+    robot_ip="$(arg ip_address)"
     namespace="$(arg namespace)"
     parent="$(arg parent)"
   />
-  <!-- realsense: -->
-  <xacro:if value="$(arg load_realsense)">
-    <xacro:include filename="$(find rcdt_sensors)/urdf/rcdt_realsense_d435.urdf.xacro" />
-    <link name="realsense_link" />
-    <joint name="realsense_link_joint" type="fixed">
-      <origin xyz="0.05 -0.02 0.01" rpy="0 ${-0.5*pi} ${pi}" />
-      <parent link="fr3_hand" />
-      <child link="realsense_link" />
-    </joint>
-    <xacro:rcdt_realsense_d435
-      robot_namespace="$(arg namespace)"
-      device_namespace="realsense"
-      parent="realsense_link"
-      gazebo="$(arg simulation)"
-    />
-  </xacro:if>
+  <!-- Create detachable joints between base_link and childs: -->
+  <xacro:include filename="$(find rcdt_utilities)/urdf/detachable_joints.urdf.xacro" />
+  <xacro:detachable_joints parent_link="fr3_link0" childs="${$(arg childs)}" />
 </robot>

File: ros2_ws/src/rcdt_sensors/urdf/rcdt_velodyne.urdf.xacro (robot description, xacro)
@@ -15,4 +15,5 @@
     *origin
     namespace
+    parent
     name:=velodyne
     update_rate:=10
@@ -67,4 +68,14 @@
       </visual>
     </link>
+    <!-- Gazebo requires a joint to a link called "world" for statically mounted robots -->
+    <xacro:if value="${parent != ''}">
+      <xacro:if value="${parent == 'world'}">
+        <link name="${parent}" />
+        <joint name="${parent}_joint" type="fixed">
+          <parent link="${parent}" />
+          <child link="base_link" />
+        </joint>
+      </xacro:if>
+    </xacro:if>
     <gazebo reference="${name}">
       <sensor type="gpu_lidar" name="${namespace}">
@@ -104,5 +115,7 @@
     </gazebo>
   </xacro:macro>
-  <xacro:VLP-16 namespace="velodyne">
+  <xacro:arg name="namespace" default="velodyne" />
+  <xacro:arg name="parent" default="" />
+  <xacro:VLP-16 namespace="$(arg namespace)" parent="$(arg parent)">
     <origin xyz="0 0 0" rpy="0 0 0" />
   </xacro:VLP-16>

Commit message: Add support for other links and orientations.
Signed-off-by: Jelmer de Wolde <jelmer.de.wolde@alliander.com>

File: ros2_ws/src/rcdt_franka/urdf/franka.urdf.xacro (robot description, xacro)
@@ -36,6 +36,10 @@
     parent="$(arg parent)"
   />
-  <!-- Create detachable joints between base_link and childs: -->
+  <!-- Preserve joint so that child link can be used for detachable joints: -->
+  <gazebo reference="fr3_hand_joint">
+    <preserveFixedJoint>true</preserveFixedJoint>
+  </gazebo>
+  <!-- Create detachable joints with given childs: -->
   <xacro:include filename="$(find rcdt_utilities)/urdf/detachable_joints.urdf.xacro" />
-  <xacro:detachable_joints parent_link="fr3_link0" childs="${$(arg childs)}" />
+  <xacro:detachable_joints childs="${$(arg childs)}" />
 </robot>

File: ros2_ws/src/rcdt_panther/urdf/panther.urdf.xacro (robot description, xacro)
@@ -18,6 +18,6 @@
     battery_config_file=""
     namespace="$(arg namespace)" />
-  <!-- Create detachable joints between base_link and childs: -->
+  <!-- Create detachable joints with given childs: -->
   <xacro:include filename="$(find rcdt_utilities)/urdf/detachable_joints.urdf.xacro" />
-  <xacro:detachable_joints parent_link="base_link" childs="${$(arg childs)}" />
+  <xacro:detachable_joints childs="${$(arg childs)}" />
 </robot>

File: ros2_ws/src/rcdt_utilities/urdf/detachable_joints.urdf.xacro (robot description, xacro)
@@ -5,5 +5,5 @@
 -->
 <robot xmlns:xacro="http://wiki.ros.org/xacro">
-  <xacro:macro name="detachable_joints" params="parent_link:=^ childs:=^">
+  <xacro:macro name="detachable_joints" params="childs:=^">
     <xacro:if value="${childs}">
       <!-- Select the child from the list: -->
@@ -11,6 +11,7 @@
       <!-- If child is not empty, select the model and link names: -->
       <xacro:if value="${child}">
-        <xacro:property name="model" value="${child.pop(0)}" />
-        <xacro:property name="link" value="${child.pop(0)}" />
+        <xacro:property name="parent_link" value="${child.pop(0)}" />
+        <xacro:property name="child_model" value="${child.pop(0)}" />
+        <xacro:property name="child_link" value="${child.pop(0)}" />
         <!-- Create the detachable joint: -->
         <gazebo>
@@ -18,6 +19,6 @@
             name="gz::sim::systems::DetachableJoint">
             <parent_link>${parent_link}</parent_link>
-            <child_model>${model}</child_model>
-            <child_link>${link}</child_link>
+            <child_model>${child_model}</child_model>
+            <child_link>${child_link}</child_link>
           </plugin>
         </gazebo>
