Commit message: Update Franka URDFs.
Signed-off-by: Jelmer de Wolde <jelmer.de.wolde@alliander.com>

File: ros2_ws/src/rcdt_franka/urdf/adapted/franka_arm.ros2_control.xacro (robot description, xacro)
@@ -2,5 +2,5 @@
 <!--
 Based on:
-https://github.com/frankaemika/franka_description/blob/0.4.0/robots/common/franka_arm.ros2_control.xacro
+https://github.com/frankarobotics/franka_description/blob/1.0.1/robots/common/franka_arm.ros2_control.xacro
 A copy of the original file is located in the /original directory.
 To compare the two files in VSCode, see:
@@ -10,16 +10,16 @@
 <xacro:macro name="franka_arm_ros2_control"
          params="arm_id
-             robot_ip
-             use_fake_hardware:=^|false
-             fake_sensor_commands:=^|false
-             gazebo:=^|false
-             hand:=^|false
-             gazebo_effort:=^|false
-             arm_prefix:=''
-             multi_arm:=false
-             namespace:=''">
+                 robot_ip
+                 use_fake_hardware:=false
+                 fake_sensor_commands:=false
+                 gazebo:=false
+                 hand:=false
+                 gazebo_effort:=false
+                 arm_prefix:=''
+                 namespace:=''">
     <xacro:property name="arm_prefix_modified" value="${'' if arm_prefix == '' else arm_prefix + '_'}" />
     <ros2_control name="${arm_prefix_modified}FrankaHardwareInterface" type="system">
         <hardware>
+          <param name="version">0.1.0</param>
           <param name="arm_id">${arm_id}</param>
           <param name="prefix">${arm_prefix}</param>
@@ -32,16 +32,11 @@
             <plugin>gz_ros2_control/GazeboSimSystem</plugin>
           </xacro:if>
-          <xacro:if value="${use_fake_hardware == 0 and gazebo == 0 and multi_arm == 0}">
+          <xacro:if value="${use_fake_hardware == 0 and gazebo == 0}">
             <plugin>franka_hardware/FrankaHardwareInterface</plugin>
-            <param name="robot_ip">${robot_ip}</param>
-            <param name="arm_prefix">${arm_prefix}</param>
-            <param name="version">0.0.0</param>
-          </xacro:if>
-          <xacro:if value="${use_fake_hardware == 0 and gazebo == 0 and multi_arm == 1}">
-            <plugin>franka_hardware/MultiFrankaHardwareInterface</plugin>
             <param name="robot_ip">${robot_ip}</param>
             <param name="arm_prefix">${arm_prefix}</param>
           </xacro:if>
         </hardware>
+      <!-- Joint position, velocity and effort interfaces -->
       <xacro:macro name="configure_joint" params="joint_name initial_position">
         <joint name="${joint_name}">
@@ -50,8 +45,6 @@
             https://github.com/ros-controls/gz_ros2_control/issues/343
             Command Interfaces -->
-          <xacro:if value="${multi_arm == 0}">
             <command_interface name="position"/>
             <command_interface name="velocity"/>
-          </xacro:if>
           <xacro:if value="${gazebo == 0 or gazebo_effort == 1}">
             <command_interface name="effort"/>
@@ -66,11 +59,11 @@
         </joint>
       </xacro:macro>
-      <xacro:configure_joint joint_name="${arm_prefix_modified}${arm_id}_joint1" initial_position="0.0"/>
-      <xacro:configure_joint joint_name="${arm_prefix_modified}${arm_id}_joint2" initial_position="${-pi/4}"/>
-      <xacro:configure_joint joint_name="${arm_prefix_modified}${arm_id}_joint3" initial_position="0.0"/>
-      <xacro:configure_joint joint_name="${arm_prefix_modified}${arm_id}_joint4" initial_position="${-3*pi/4}"/>
-      <xacro:configure_joint joint_name="${arm_prefix_modified}${arm_id}_joint5" initial_position="0.0"/>
-      <xacro:configure_joint joint_name="${arm_prefix_modified}${arm_id}_joint6" initial_position="${pi/2}"/>
-      <xacro:configure_joint joint_name="${arm_prefix_modified}${arm_id}_joint7" initial_position="${pi/4}"/>
+      <xacro:configure_joint joint_name="${arm_prefix}${arm_id}_joint1" initial_position="0.0"/>
+      <xacro:configure_joint joint_name="${arm_prefix}${arm_id}_joint2" initial_position="${-pi/4}"/>
+      <xacro:configure_joint joint_name="${arm_prefix}${arm_id}_joint3" initial_position="0.0"/>
+      <xacro:configure_joint joint_name="${arm_prefix}${arm_id}_joint4" initial_position="${-3*pi/4}"/>
+      <xacro:configure_joint joint_name="${arm_prefix}${arm_id}_joint5" initial_position="0.0"/>
+      <xacro:configure_joint joint_name="${arm_prefix}${arm_id}_joint6" initial_position="${pi/2}"/>
+      <xacro:configure_joint joint_name="${arm_prefix}${arm_id}_joint7" initial_position="${pi/4}"/>
       <xacro:if value="${gazebo and hand}">
         <xacro:configure_joint joint_name="${arm_id}_finger_joint1" initial_position="0.0" />
@@ -81,4 +74,28 @@
         </joint>
       </xacro:if>
+      <xacro:macro name="general_purpose_io" params="prefix command_interface index">
+        <gpio name="${prefix}">
+          <command_interface name="${command_interface}"/>
+          <param name="index">${index}</param>
+        </gpio>
+      </xacro:macro>
+      <!-- Cartesian velocity interfaces -->
+      <xacro:general_purpose_io prefix="vx" command_interface="cartesian_velocity" index="0"/>
+      <xacro:general_purpose_io prefix="vy" command_interface="cartesian_velocity" index="1"/>
+      <xacro:general_purpose_io prefix="vz" command_interface="cartesian_velocity" index="2"/>
+      <xacro:general_purpose_io prefix="wx" command_interface="cartesian_velocity" index="3"/>
+      <xacro:general_purpose_io prefix="wy" command_interface="cartesian_velocity" index="4"/>
+      <xacro:general_purpose_io prefix="wz" command_interface="cartesian_velocity" index="5"/>
+      <!-- Cartesian pose interfaces, in total 16 interfaces -->
+      <xacro:macro name="loop" params="i">
+        <xacro:unless value="${i == 16}">
+          <xacro:general_purpose_io prefix="${i}" command_interface="cartesian_pose_command" index="${i}"/>
+          <xacro:loop i="${i+1}"/>
+        </xacro:unless>
+      </xacro:macro>
+      <xacro:loop i="0"/>
+      <!-- Elbow command interfaces -->
+      <xacro:general_purpose_io prefix="joint_3_position" command_interface="elbow_command" index="0"/>
+      <xacro:general_purpose_io prefix="joint_4_sign" command_interface="elbow_command" index="1"/>
     </ros2_control>
     <xacro:if value="${gazebo}">

File: ros2_ws/src/rcdt_franka/urdf/adapted/franka_robot.xacro (robot description, xacro)
@@ -2,5 +2,5 @@
 <!--
 Based on:
-https://github.com/frankaemika/franka_description/blob/0.4.0/robots/common/franka_robot.xacro
+https://github.com/frankarobotics/franka_description/blob/1.0.1/robots/common/franka_robot.xacro
 A copy of the original file is located in the /original directory.
 To compare the two files in VSCode, see:
@@ -18,6 +18,12 @@
                       xyz:='0 0 0'
                       rpy:='0 0 0'
+                      xyz_ee:='0 0 0'
+                      rpy_ee:='0 0 0'
+                      tcp_xyz:='0 0 0'
+                      tcp_rpy:='0 0 0'
+                      safety_distance:='0.03'
                       hand:='true'
                       ee_id:=none
+                      special_connection:=''
                       gazebo:='false'
                       with_sc:='false'
@@ -29,20 +35,13 @@
                       no_prefix:='false'
                       arm_prefix:=''
-                      connected_to:='base'
-                      multi_arm:=false">
+                      description_pkg:='franka_description'
+                      connected_to:='base'">
     <!-- Map params to args: -->
-    <xacro:arg name="hand" default="${hand}" />
-    <xacro:arg name="ee_id" default="${ee_id}" />
-    <xacro:arg name="gazebo" default="${gazebo}" />
-    <xacro:arg name="use_fake_hardware" default="${use_fake_hardware}" />
-    <xacro:arg name="fake_sensor_commands" default="${fake_sensor_commands}" />
-    <xacro:arg name="gazebo_effort" default="${gazebo_effort}" />
-    <xacro:arg name="multi_arm" default="${multi_arm}" />
+    <xacro:arg name="special_connection" default="${special_connection}" />
     <xacro:include filename="$(find franka_description)/robots/common/utils.xacro" />
     <xacro:include filename="$(find franka_description)/robots/common/franka_arm.xacro" />
-    <xacro:property name="arm_prefix_modified" value="${'' if arm_prefix == '' else arm_prefix + '_'}" />
     <xacro:franka_arm
       arm_id="${arm_id}"
-      arm_prefix="${arm_prefix_modified}"
+      arm_prefix="${arm_prefix}"
       no_prefix="${no_prefix}"
       xyz="${xyz}"
@@ -60,9 +59,8 @@
       <xacro:include filename="$(find franka_description)/end_effectors/common/franka_hand.xacro"/>
       <xacro:include filename="$(find franka_description)/end_effectors/common/utils.xacro" />
-      <xacro:include filename="$(find franka_description)/end_effectors/$(arg ee_id)/$(arg ee_id)_arguments.xacro" />
       <xacro:if value="${arm_id == 'fp3'}">
         <xacro:property name="ee_color" value="black" />
       </xacro:if>
-      <xacro:if value="${arm_id == 'fr3' or arm_id == 'fer'}">
+      <xacro:if value="${arm_id == 'fr3' or arm_id == 'fer' or arm_id == 'fr3v2'}">
         <xacro:property name="ee_color" value="white" />
       </xacro:if>
@@ -70,16 +68,16 @@
       <xacro:property name="connection" value="${special_connection if special_connection != '' else arm_id + '_link8'}" />
       <xacro:franka_hand
-        connected_to="${arm_prefix_modified}${connection}"
+        connected_to="${arm_prefix}${connection}"
         arm_id="${arm_id}"
-        arm_prefix="${arm_prefix_modified}"
+        arm_prefix="${arm_prefix}"
         ee_id="${ee_id}_${ee_color}"
-        ee_inertials="${xacro.load_yaml('$(find franka_description)/end_effectors/$(arg ee_id)/inertials.yaml')}"
-        rpy_ee="$(arg rpy_ee)"
-        xyz_ee="$(arg xyz_ee)"
-        tcp_xyz="$(arg tcp_xyz)"
-        tcp_rpy="$(arg tcp_rpy)"
-        safety_distance="$(arg safety_distance)"
+        ee_inertials="${xacro.load_yaml('$(find franka_description)/end_effectors/' + ee_id + '/inertials.yaml')}"
+        rpy_ee="${rpy_ee}"
+        xyz_ee="${xyz_ee}"
+        tcp_xyz="${tcp_xyz}"
+        tcp_rpy="${tcp_rpy}"
+        safety_distance="${safety_distance}"
         gazebo="${gazebo}"
-        description_pkg="$(arg description_pkg)"
+        description_pkg="${description_pkg}"
         with_sc="${with_sc}"
       />
@@ -88,20 +86,19 @@
       <xacro:include filename="$(find franka_description)/end_effectors/common/ee_with_one_link.xacro"/>
       <xacro:include filename="$(find franka_description)/end_effectors/common/utils.xacro" />
-      <xacro:include filename="$(find franka_description)/end_effectors/$(arg ee_id)/$(arg ee_id)_arguments.xacro" />
-      <xacro:property name="special_connection" value="$(arg special_connection)" />
+      <xacro:property name="special_connection" value="${special_connection}" />
       <xacro:property name="connection" value="${special_connection if special_connection == '' else arm_id + '_link8'}" />
       <xacro:ee_with_one_link
-        connected_to="${arm_prefix_modified}${connection}"
+        connected_to="${arm_prefix}${connection}"
         arm_id="${arm_id}"
-        arm_prefix="${arm_prefix_modified}"
+        arm_prefix="${arm_prefix}"
         ee_id="${ee_id}"
-        ee_inertials="${xacro.load_yaml('$(find franka_description)/end_effectors/$(arg ee_id)/inertials.yaml')}"
-        rpy_ee="$(arg rpy_ee)"
-        xyz_ee="$(arg xyz_ee)"
-        tcp_xyz="$(arg tcp_xyz)"
-        tcp_rpy="$(arg tcp_rpy)"
-        safety_distance="$(arg safety_distance)"
+        ee_inertials="${xacro.load_yaml('$(find franka_description)/end_effectors/${ee_id}/inertials.yaml')}"
+        rpy_ee="${rpy_ee}"
+        xyz_ee="${xyz_ee}"
+        tcp_xyz="${tcp_xyz}"
+        tcp_rpy="${tcp_rpy}"
+        safety_distance="${safety_distance}"
         gazebo="${gazebo}"
-        description_pkg="$(arg description_pkg)"
+        description_pkg="${description_pkg}"
         with_sc="${with_sc}"
       />
@@ -159,11 +156,10 @@
           arm_id="${arm_id}"
           robot_ip="${robot_ip}"
-          use_fake_hardware="$(arg use_fake_hardware)"
-          fake_sensor_commands="$(arg fake_sensor_commands)"
-          gazebo="$(arg gazebo)"
-          hand="$(arg hand)"
-          gazebo_effort="$(arg gazebo_effort)"
+          use_fake_hardware="${use_fake_hardware}"
+          fake_sensor_commands="${fake_sensor_commands}"
+          gazebo="${gazebo}"
+          hand="${hand}"
+          gazebo_effort="${gazebo_effort}"
           arm_prefix="${arm_prefix}"
-          multi_arm="$(arg multi_arm)"
       />
     </xacro:if>

File: ros2_ws/src/rcdt_franka/urdf/franka.urdf.xacro (robot description, xacro)
@@ -5,5 +5,11 @@
 -->
 <robot xmlns:xacro="http://www.ros.org/wiki/xacro" name="franka">
-  <!-- arguments: -->
+  <!-- Arguments from Franka, based on: -->
+  <!-- https://github.com/frankarobotics/franka_description/blob/1.0.1/robots/fr3/fr3.urdf.xacro -->
+  <xacro:arg name="xyz_ee" default="0 0 0" />
+  <xacro:arg name="rpy_ee" default="0 0 ${-pi/4}" />
+  <xacro:arg name="tcp_xyz" default="0 0 0.1034" />
+  <xacro:arg name="tcp_rpy" default="0 0 0" />
+  <!-- Custom arguments: -->
   <xacro:arg name="namespace" default="" />
   <xacro:arg name="simulation" default="false" />
@@ -14,13 +20,17 @@
   <xacro:franka_robot
     arm_id="fr3"
-    ee_id="franka_hand"
-    ros2_control="true"
-    robot_ip="10.15.20.4"
     joint_limits="${xacro.load_yaml('$(find franka_description)/robots/fr3/joint_limits.yaml')}"
     inertials="${xacro.load_yaml('$(find franka_description)/robots/fr3/inertials.yaml')}"
     kinematics="${xacro.load_yaml('$(find franka_description)/robots/fr3/kinematics.yaml')}"
     dynamics="${xacro.load_yaml('$(find franka_description)/robots/fr3/dynamics.yaml')}"
+    gazebo="$(arg simulation)"
+    ee_id="franka_hand"
+    xyz_ee="$(arg xyz_ee)"
+    rpy_ee="$(arg rpy_ee)"
+    tcp_xyz="$(arg tcp_xyz)"
+    tcp_rpy="$(arg tcp_rpy)"
+    ros2_control="true"
+    robot_ip="10.15.20.4"
     namespace="$(arg namespace)"
-    gazebo="$(arg simulation)"
     parent="$(arg parent)"
   />

File: ros2_ws/src/rcdt_franka/urdf/original/franka_arm.ros2_control.xacro (robot description, xacro)
@@ -3,15 +3,15 @@
 <xacro:macro name="franka_arm_ros2_control"
          params="arm_id
-             robot_ip
-             use_fake_hardware:=^|false
-             fake_sensor_commands:=^|false
-             gazebo:=^|false
-             hand:=^|false
-             gazebo_effort:=^|false
-             arm_prefix:=''
-             multi_arm:=false">
+                 robot_ip
+                 use_fake_hardware:=false
+                 fake_sensor_commands:=false
+                 gazebo:=false
+                 hand:=false
+                 gazebo_effort:=false
+                 arm_prefix:=''">
     <xacro:property name="arm_prefix_modified" value="${'' if arm_prefix == '' else arm_prefix + '_'}" />
     <ros2_control name="${arm_prefix_modified}FrankaHardwareInterface" type="system">
         <hardware>
+          <param name="version">0.1.0</param>
           <param name="arm_id">${arm_id}</param>
           <param name="prefix">${arm_prefix}</param>
@@ -24,15 +24,11 @@
             <plugin>franka_ign_ros2_control/IgnitionSystem</plugin>
           </xacro:if>
-          <xacro:if value="${use_fake_hardware == 0 and gazebo == 0 and multi_arm == 0}">
+          <xacro:if value="${use_fake_hardware == 0 and gazebo == 0}">
             <plugin>franka_hardware/FrankaHardwareInterface</plugin>
             <param name="robot_ip">${robot_ip}</param>
             <param name="arm_prefix">${arm_prefix}</param>
           </xacro:if>
-          <xacro:if value="${use_fake_hardware == 0 and gazebo == 0 and multi_arm == 1}">
-            <plugin>franka_hardware/MultiFrankaHardwareInterface</plugin>
-            <param name="robot_ip">${robot_ip}</param>
-            <param name="arm_prefix">${arm_prefix}</param>
-          </xacro:if>
         </hardware>
+      <!-- Joint position, velocity and effort interfaces -->
       <xacro:macro name="configure_joint" params="joint_name initial_position">
         <joint name="${joint_name}">
@@ -41,8 +37,6 @@
             https://github.com/ros-controls/gz_ros2_control/issues/343
             Command Interfaces -->
-          <xacro:if value="${multi_arm == 0}">
             <command_interface name="position"/>
             <command_interface name="velocity"/>
-          </xacro:if>
           <xacro:if value="${gazebo == 0 or gazebo_effort == 1}">
             <command_interface name="effort"/>
@@ -57,14 +51,38 @@
         </joint>
       </xacro:macro>
-      <xacro:configure_joint joint_name="${arm_prefix_modified}${arm_id}_joint1" initial_position="0.0"/>
-      <xacro:configure_joint joint_name="${arm_prefix_modified}${arm_id}_joint2" initial_position="${-pi/4}"/>
-      <xacro:configure_joint joint_name="${arm_prefix_modified}${arm_id}_joint3" initial_position="0.0"/>
-      <xacro:configure_joint joint_name="${arm_prefix_modified}${arm_id}_joint4" initial_position="${-3*pi/4}"/>
-      <xacro:configure_joint joint_name="${arm_prefix_modified}${arm_id}_joint5" initial_position="0.0"/>
-      <xacro:configure_joint joint_name="${arm_prefix_modified}${arm_id}_joint6" initial_position="${pi/2}"/>
-      <xacro:configure_joint joint_name="${arm_prefix_modified}${arm_id}_joint7" initial_position="${pi/4}"/>
+      <xacro:configure_joint joint_name="${arm_prefix}${arm_id}_joint1" initial_position="0.0"/>
+      <xacro:configure_joint joint_name="${arm_prefix}${arm_id}_joint2" initial_position="${-pi/4}"/>
+      <xacro:configure_joint joint_name="${arm_prefix}${arm_id}_joint3" initial_position="0.0"/>
+      <xacro:configure_joint joint_name="${arm_prefix}${arm_id}_joint4" initial_position="${-3*pi/4}"/>
+      <xacro:configure_joint joint_name="${arm_prefix}${arm_id}_joint5" initial_position="0.0"/>
+      <xacro:configure_joint joint_name="${arm_prefix}${arm_id}_joint6" initial_position="${pi/2}"/>
+      <xacro:configure_joint joint_name="${arm_prefix}${arm_id}_joint7" initial_position="${pi/4}"/>
       <xacro:if value="${gazebo and hand}">
         <xacro:configure_joint joint_name="${arm_id}_finger_joint1" initial_position="0.0" />
       </xacro:if>
+      <xacro:macro name="general_purpose_io" params="prefix command_interface index">
+        <gpio name="${prefix}">
+          <command_interface name="${command_interface}"/>
+          <param name="index">${index}</param>
+        </gpio>
+      </xacro:macro>
+      <!-- Cartesian velocity interfaces -->
+      <xacro:general_purpose_io prefix="vx" command_interface="cartesian_velocity" index="0"/>
+      <xacro:general_purpose_io prefix="vy" command_interface="cartesian_velocity" index="1"/>
+      <xacro:general_purpose_io prefix="vz" command_interface="cartesian_velocity" index="2"/>
+      <xacro:general_purpose_io prefix="wx" command_interface="cartesian_velocity" index="3"/>
+      <xacro:general_purpose_io prefix="wy" command_interface="cartesian_velocity" index="4"/>
+      <xacro:general_purpose_io prefix="wz" command_interface="cartesian_velocity" index="5"/>
+      <!-- Cartesian pose interfaces, in total 16 interfaces -->
+      <xacro:macro name="loop" params="i">
+        <xacro:unless value="${i == 16}">
+          <xacro:general_purpose_io prefix="${i}" command_interface="cartesian_pose_command" index="${i}"/>
+          <xacro:loop i="${i+1}"/>
+        </xacro:unless>
+      </xacro:macro>
+      <xacro:loop i="0"/>
+      <!-- Elbow command interfaces -->
+      <xacro:general_purpose_io prefix="joint_3_position" command_interface="elbow_command" index="0"/>
+      <xacro:general_purpose_io prefix="joint_4_sign" command_interface="elbow_command" index="1"/>
     </ros2_control>
     <xacro:if value="${gazebo}">
