Commit message: Move panther and lynx to new husarion package, as well as the corresponding controller config from rcdt_gazebo
Signed-off-by: Rosalie <rosalie.van.ark@alliander.com>

File: ros2_ws/src/rcdt_husarion/urdf/lynx/adapted/lynx_macro.urdf.xacro (robot description, xacro)
@@ -2,5 +2,5 @@
 <!--
 Based on:
-https://github.com/husarion/husarion_ugv_ros/blob/2.3.1/husarion_ugv_description/urdf/panther/panther_macro.urdf.xacro
+https://github.com/husarion/husarion_ugv_ros/blob/2.3.1/husarion_ugv_description/urdf/lynx/lynx_macro.urdf.xacro
 A copy of the original file is located in the /original directory.
 To compare the two files in VSCode, see:
@@ -9,23 +9,23 @@
 <robot xmlns:xacro="http://wiki.ros.org/xacro">
   <xacro:macro
-    name="panther_robot"
+    name="lynx_robot"
     params="wheel_config_file
             controller_config_file
             battery_config_file
             use_sim:=false
-            imu_xyz:='0.169 0.025 0.092'
+            imu_xyz:='0.052 0.073 -0.006'
             imu_rpy:='0.0 0.0 -1.57'
             namespace:=''">
     <xacro:if value="${use_sim}">
-      <xacro:property name="imu_xyz" value="-0.195 0.010 0.085" />
-      <xacro:property name="imu_rpy" value="0.000 -0.000 3.142" />
+      <xacro:property name="imu_xyz" value="0.052 0.073 -0.006" />
+      <xacro:property name="imu_rpy" value="0.0 0.0 -1.57" />
     </xacro:if>
     <xacro:property name="ns" value='${namespace + "/" if namespace else ""}' />
     <xacro:property name="wheel_config" value="${xacro.load_yaml(wheel_config_file)}" />
-    <xacro:property name="wheelbase" value="0.44" />
-    <xacro:property name="wheel_mount_point_y" value="0.2575" />
+    <xacro:property name="wheelbase" value="0.35" />
+    <xacro:property name="wheel_mount_point_y" value="0.1675" />
     <!-- INCLUDE ROBOT PARTS DEFINITIONS -->
-    <xacro:include filename="$(find husarion_ugv_description)/urdf/panther/base.urdf.xacro" ns="body" />
-    <xacro:include filename="$(find rcdt_panther)/urdf/adapted/gazebo.urdf.xacro" ns="gazebo" />
+    <xacro:include filename="$(find husarion_ugv_description)/urdf/lynx/base.urdf.xacro" ns="body" />
+    <xacro:include filename="$(find rcdt_husarion)/urdf/lynx/adapted/gazebo.urdf.xacro" ns="gazebo" />
     <xacro:include filename="$(find husarion_ugv_description)/urdf/common/wheel.urdf.xacro" ns="wheel" />
     <!-- BODY DECLARATION -->
@@ -55,5 +55,5 @@
       mount_point_y="${wheel_mount_point_y}"
       prefix="rr" />
-    <ros2_control name="${ns}panther_system" type="system">
+    <ros2_control name="${ns}lynx_system" type="system">
       <hardware>
         <xacro:if value="${use_sim}">
@@ -61,5 +61,5 @@
         </xacro:if>
         <xacro:unless value="${use_sim}">
-          <plugin>husarion_ugv_hardware_interfaces/PantherSystem</plugin>
+          <plugin>husarion_ugv_hardware_interfaces/LynxSystem</plugin>
           <param name="encoder_resolution">1600</param>
           <param name="gear_ratio">30.08</param>
@@ -71,6 +71,5 @@
           <param name="can_interface_name">robot_can</param>
           <param name="master_can_id">3</param>
-          <param name="front_driver_can_id">1</param>
-          <param name="rear_driver_can_id">2</param>
+          <param name="driver_can_id">1</param>
           <param name="sdo_operation_timeout_ms">100</param>
           <!-- Depends on frequency of the controller, more critical motors state are sent with
@@ -167,6 +166,7 @@
       <xacro:gazebo.controller config_file="${controller_config_file}" namespace="${namespace}" />
       <xacro:gazebo.imu reference_frame="imu_link" namespace="${namespace}" />
-      <xacro:gazebo.light reference_frame="lights_channel_1_link" name="lights_channel_1" topic="lights/channel_1_frame" namespace="${namespace}" />
-      <xacro:gazebo.light reference_frame="lights_channel_2_link" name="lights_channel_2" topic="lights/channel_2_frame" namespace="${namespace}" />
+      <!-- TODO Add lights visualization -->
+      <!-- <xacro:gazebo.light reference_frame="lights_channel_1_link" name="lights_channel_1" topic="lights/channel_1_frame" namespace="${namespace}" /> -->
+      <!-- <xacro:gazebo.light reference_frame="lights_channel_2_link" name="lights_channel_2" topic="lights/channel_2_frame" namespace="${namespace}" /> -->
     </xacro:if>
   </xacro:macro>

File: ros2_ws/src/rcdt_husarion/urdf/lynx/lynx.urdf.xacro (robot description, xacro)
@@ -12,5 +12,5 @@
   <xacro:arg name="childs" default="${[]}" />
   <!-- Load lynx: -->
-  <xacro:include filename="$(find rcdt_lynx)/urdf/adapted/lynx_macro.urdf.xacro" ns="husarion" />
+  <xacro:include filename="$(find rcdt_husarion)/urdf/lynx/adapted/lynx_macro.urdf.xacro" ns="husarion" />
   <xacro:husarion.lynx_robot
     use_sim="$(arg use_sim)"
@@ -18,5 +18,5 @@
     imu_rpy="$(arg imu_rpy)"
     wheel_config_file="$(find husarion_ugv_description)/config/WH05.yaml"
-    controller_config_file="$(find rcdt_gazebo)/config/controllers.yaml"
+    controller_config_file="$(find rcdt_husarion)/config/lynx_controllers.yaml"
     battery_config_file=""
     namespace="$(arg namespace)" />

File: ros2_ws/src/rcdt_husarion/urdf/panther/adapted/panther_macro.urdf.xacro (robot description, xacro)
@@ -2,5 +2,5 @@
 <!--
 Based on:
-https://github.com/husarion/husarion_ugv_ros/blob/2.3.1/husarion_ugv_description/urdf/lynx/lynx_macro.urdf.xacro
+https://github.com/husarion/husarion_ugv_ros/blob/2.3.1/husarion_ugv_description/urdf/panther/panther_macro.urdf.xacro
 A copy of the original file is located in the /original directory.
 To compare the two files in VSCode, see:
@@ -9,23 +9,23 @@
 <robot xmlns:xacro="http://wiki.ros.org/xacro">
   <xacro:macro
-    name="lynx_robot"
+    name="panther_robot"
     params="wheel_config_file
             controller_config_file
             battery_config_file
             use_sim:=false
-            imu_xyz:='0.052 0.073 -0.006'
+            imu_xyz:='0.169 0.025 0.092'
             imu_rpy:='0.0 0.0 -1.57'
             namespace:=''">
     <xacro:if value="${use_sim}">
-      <xacro:property name="imu_xyz" value="0.052 0.073 -0.006" />
-      <xacro:property name="imu_rpy" value="0.0 0.0 -1.57" />
+      <xacro:property name="imu_xyz" value="-0.195 0.010 0.085" />
+      <xacro:property name="imu_rpy" value="0.000 -0.000 3.142" />
     </xacro:if>
     <xacro:property name="ns" value='${namespace + "/" if namespace else ""}' />
     <xacro:property name="wheel_config" value="${xacro.load_yaml(wheel_config_file)}" />
-    <xacro:property name="wheelbase" value="0.35" />
-    <xacro:property name="wheel_mount_point_y" value="0.1675" />
+    <xacro:property name="wheelbase" value="0.44" />
+    <xacro:property name="wheel_mount_point_y" value="0.2575" />
     <!-- INCLUDE ROBOT PARTS DEFINITIONS -->
-    <xacro:include filename="$(find husarion_ugv_description)/urdf/lynx/base.urdf.xacro" ns="body" />
-    <xacro:include filename="$(find rcdt_lynx)/urdf/adapted/gazebo.urdf.xacro" ns="gazebo" />
+    <xacro:include filename="$(find husarion_ugv_description)/urdf/panther/base.urdf.xacro" ns="body" />
+    <xacro:include filename="$(find rcdt_husarion)/urdf/panther/adapted/gazebo.urdf.xacro" ns="gazebo" />
     <xacro:include filename="$(find husarion_ugv_description)/urdf/common/wheel.urdf.xacro" ns="wheel" />
     <!-- BODY DECLARATION -->
@@ -55,5 +55,5 @@
       mount_point_y="${wheel_mount_point_y}"
       prefix="rr" />
-    <ros2_control name="${ns}lynx_system" type="system">
+    <ros2_control name="${ns}panther_system" type="system">
       <hardware>
         <xacro:if value="${use_sim}">
@@ -61,5 +61,5 @@
         </xacro:if>
         <xacro:unless value="${use_sim}">
-          <plugin>husarion_ugv_hardware_interfaces/LynxSystem</plugin>
+          <plugin>husarion_ugv_hardware_interfaces/PantherSystem</plugin>
           <param name="encoder_resolution">1600</param>
           <param name="gear_ratio">30.08</param>
@@ -71,5 +71,6 @@
           <param name="can_interface_name">robot_can</param>
           <param name="master_can_id">3</param>
-          <param name="driver_can_id">1</param>
+          <param name="front_driver_can_id">1</param>
+          <param name="rear_driver_can_id">2</param>
           <param name="sdo_operation_timeout_ms">100</param>
           <!-- Depends on frequency of the controller, more critical motors state are sent with
@@ -166,7 +167,6 @@
       <xacro:gazebo.controller config_file="${controller_config_file}" namespace="${namespace}" />
       <xacro:gazebo.imu reference_frame="imu_link" namespace="${namespace}" />
-      <!-- TODO Add lights visualization -->
-      <!-- <xacro:gazebo.light reference_frame="lights_channel_1_link" name="lights_channel_1" topic="lights/channel_1_frame" namespace="${namespace}" /> -->
-      <!-- <xacro:gazebo.light reference_frame="lights_channel_2_link" name="lights_channel_2" topic="lights/channel_2_frame" namespace="${namespace}" /> -->
+      <xacro:gazebo.light reference_frame="lights_channel_1_link" name="lights_channel_1" topic="lights/channel_1_frame" namespace="${namespace}" />
+      <xacro:gazebo.light reference_frame="lights_channel_2_link" name="lights_channel_2" topic="lights/channel_2_frame" namespace="${namespace}" />
     </xacro:if>
   </xacro:macro>

File: ros2_ws/src/rcdt_husarion/urdf/panther/panther.urdf.xacro (robot description, xacro)
@@ -10,10 +10,10 @@
   <xacro:arg name="childs" default="${[]}" />
   <!-- Load panther: -->
-  <xacro:include filename="$(find rcdt_panther)/urdf/adapted/panther_macro.urdf.xacro"
+  <xacro:include filename="$(find rcdt_husarion)/urdf/panther/adapted/panther_macro.urdf.xacro"
     ns="husarion" />
   <xacro:husarion.panther_robot
     use_sim="$(arg simulation)"
     wheel_config_file="$(find husarion_ugv_description)/config/WH01.yaml"
-    controller_config_file="$(find rcdt_gazebo)/config/controllers.yaml"
+    controller_config_file="$(find rcdt_husarion)/config/panther_controllers.yaml"
     battery_config_file=""
     namespace="$(arg namespace)" />

Commit message: 289 lynx integrate lynx simulation (#351)
* Add lynx startup to repo, only in rviz the link to map not working yet

Signed-off-by: Rosalie <rosalie.van.ark@alliander.com>

* Adjust controller config location in urdf lynx, but it's the panther version so the lynx version still needs to be added!

Signed-off-by: Rosalie <rosalie.van.ark@alliander.com>

* Fix linting

Signed-off-by: Rosalie <rosalie.van.ark@alliander.com>

* Move panther and lynx to new husarion package, as well as the corresponding controller config from rcdt_gazebo

Signed-off-by: Rosalie <rosalie.van.ark@alliander.com>

* Restore removed config value

Signed-off-by: Rosalie <rosalie.van.ark@alliander.com>

* Move the nav2 parts from the panther package to its own package

Signed-off-by: Rosalie <rosalie.van.ark@alliander.com>

* Add ouster lidar and gps configurations, tested via bringup

Signed-off-by: Rosalie <rosalie.van.ark@alliander.com>

* Fix linting and add Lynx tests

Signed-off-by: Rosalie <rosalie.van.ark@alliander.com>

* Update documentation

Signed-off-by: Rosalie <rosalie.van.ark@alliander.com>

* Remove joy_topics.yaml seems it does not seem to be used anymore

Signed-off-by: Rosalie <rosalie.van.ark@alliander.com>

* Move the gazebo.urdf.xacro files to a common folder since the panther and lynx both use the same

Signed-off-by: Rosalie <rosalie.van.ark@alliander.com>

* Fix bug in nav2 tests

Signed-off-by: Rosalie <rosalie.van.ark@alliander.com>

* Add missing license file

Signed-off-by: Rosalie <rosalie.van.ark@alliander.com>

* Update predefined configurations according to new features from main branch

Signed-off-by: Rosalie <rosalie.van.ark@alliander.com>

* Fix bug regarding local variable being uninitialized

Signed-off-by: Rosalie <rosalie.van.ark@alliander.com>

* Update lifecycle node management nav2

Signed-off-by: Rosalie <rosalie.van.ark@alliander.com>

* Assign Lifecycle directly to dictionary

Signed-off-by: Rosalie <rosalie.van.ark@alliander.com>

---------

Signed-off-by: Rosalie <rosalie.van.ark@alliander.com>
Signed-off-by: Jelmer de Wolde <jelmer.de.wolde@alliander.com>
Signed-off-by: Rosalie van Ark <57712550+rosalievanark@users.noreply.github.com>
Co-authored-by: Jelmer de Wolde <jelmer.de.wolde@alliander.com>

File: ros2_ws/src/rcdt_husarion/urdf/lynx/adapted/lynx_macro.urdf.xacro (robot description, xacro)
@@ -2,5 +2,5 @@
 <!--
 Based on:
-https://github.com/husarion/husarion_ugv_ros/blob/2.3.1/husarion_ugv_description/urdf/panther/panther_macro.urdf.xacro
+https://github.com/husarion/husarion_ugv_ros/blob/2.3.1/husarion_ugv_description/urdf/lynx/lynx_macro.urdf.xacro
 A copy of the original file is located in the /original directory.
 To compare the two files in VSCode, see:
@@ -9,23 +9,23 @@
 <robot xmlns:xacro="http://wiki.ros.org/xacro">
   <xacro:macro
-    name="panther_robot"
+    name="lynx_robot"
     params="wheel_config_file
             controller_config_file
             battery_config_file
             use_sim:=false
-            imu_xyz:='0.169 0.025 0.092'
+            imu_xyz:='0.052 0.073 -0.006'
             imu_rpy:='0.0 0.0 -1.57'
             namespace:=''">
     <xacro:if value="${use_sim}">
-      <xacro:property name="imu_xyz" value="-0.195 0.010 0.085" />
-      <xacro:property name="imu_rpy" value="0.000 -0.000 3.142" />
+      <xacro:property name="imu_xyz" value="0.052 0.073 -0.006" />
+      <xacro:property name="imu_rpy" value="0.0 0.0 -1.57" />
     </xacro:if>
     <xacro:property name="ns" value='${namespace + "/" if namespace else ""}' />
     <xacro:property name="wheel_config" value="${xacro.load_yaml(wheel_config_file)}" />
-    <xacro:property name="wheelbase" value="0.44" />
-    <xacro:property name="wheel_mount_point_y" value="0.2575" />
+    <xacro:property name="wheelbase" value="0.35" />
+    <xacro:property name="wheel_mount_point_y" value="0.1675" />
     <!-- INCLUDE ROBOT PARTS DEFINITIONS -->
-    <xacro:include filename="$(find husarion_ugv_description)/urdf/panther/base.urdf.xacro" ns="body" />
-    <xacro:include filename="$(find rcdt_panther)/urdf/adapted/gazebo.urdf.xacro" ns="gazebo" />
+    <xacro:include filename="$(find husarion_ugv_description)/urdf/lynx/base.urdf.xacro" ns="body" />
+    <xacro:include filename="$(find rcdt_husarion)/urdf/common/adapted/gazebo.urdf.xacro" ns="gazebo" />
     <xacro:include filename="$(find husarion_ugv_description)/urdf/common/wheel.urdf.xacro" ns="wheel" />
     <!-- BODY DECLARATION -->
@@ -55,5 +55,5 @@
       mount_point_y="${wheel_mount_point_y}"
       prefix="rr" />
-    <ros2_control name="${ns}panther_system" type="system">
+    <ros2_control name="${ns}lynx_system" type="system">
       <hardware>
         <xacro:if value="${use_sim}">
@@ -61,5 +61,5 @@
         </xacro:if>
         <xacro:unless value="${use_sim}">
-          <plugin>husarion_ugv_hardware_interfaces/PantherSystem</plugin>
+          <plugin>husarion_ugv_hardware_interfaces/LynxSystem</plugin>
           <param name="encoder_resolution">1600</param>
           <param name="gear_ratio">30.08</param>
@@ -71,6 +71,5 @@
           <param name="can_interface_name">robot_can</param>
           <param name="master_can_id">3</param>
-          <param name="front_driver_can_id">1</param>
-          <param name="rear_driver_can_id">2</param>
+          <param name="driver_can_id">1</param>
           <param name="sdo_operation_timeout_ms">100</param>
           <!-- Depends on frequency of the controller, more critical motors state are sent with
@@ -167,6 +166,7 @@
       <xacro:gazebo.controller config_file="${controller_config_file}" namespace="${namespace}" />
       <xacro:gazebo.imu reference_frame="imu_link" namespace="${namespace}" />
-      <xacro:gazebo.light reference_frame="lights_channel_1_link" name="lights_channel_1" topic="lights/channel_1_frame" namespace="${namespace}" />
-      <xacro:gazebo.light reference_frame="lights_channel_2_link" name="lights_channel_2" topic="lights/channel_2_frame" namespace="${namespace}" />
+      <!-- TODO Add lights visualization -->
+      <!-- <xacro:gazebo.light reference_frame="lights_channel_1_link" name="lights_channel_1" topic="lights/channel_1_frame" namespace="${namespace}" /> -->
+      <!-- <xacro:gazebo.light reference_frame="lights_channel_2_link" name="lights_channel_2" topic="lights/channel_2_frame" namespace="${namespace}" /> -->
     </xacro:if>
   </xacro:macro>
