Commit message: Fix support for alliander_gui.
Signed-off-by: Jelmer de Wolde <jelmer.de.wolde@alliander.com>

File: alliander_robotics/alliander_core/src/alliander_description/ur/urdf/ur.urdf.xacro (robot description, xacro)
@@ -20,3 +20,10 @@
   <xacro:include filename="$(find alliander_utilities)/urdf/detachable_joints.urdf.xacro" />
   <xacro:detachable_joints childs="${$(arg childs)}" />
+  <!-- Create tcp link: -->
+  <link name="tcp" />
+  <joint name="tcp_joint" type="fixed">
+    <origin xyz="0 0 0" rpy="3.1416 0 0" />
+    <parent link="tool0" />
+    <child link="tcp" />
+  </joint>
 </robot>
