Commit message: 398 integrate new ur arm (#410)
* A start to bringing UR to simulation, joint state broadcaster not working yet, so the individual arm parts are not connected yet

Signed-off-by: Rosalie <rosalie.van.ark@alliander.com>

* Start UR in Gazebo with joint_state_broadcaster and joint_trajectory_controller.

Signed-off-by: Jelmer de Wolde <jelmer.de.wolde@alliander.com>

* Integrate Moveit and UR.

Signed-off-by: Jelmer de Wolde <jelmer.de.wolde@alliander.com>

* Let joystick support Franka and UR.

Signed-off-by: Jelmer de Wolde <jelmer.de.wolde@alliander.com>

* Move general MoveIt config files to general config folder.

Signed-off-by: Jelmer de Wolde <jelmer.de.wolde@alliander.com>

* Add support for child platforms connected to UR arm.

Signed-off-by: Jelmer de Wolde <jelmer.de.wolde@alliander.com>

* Add support to connect UR arm to parent platform.

Signed-off-by: Jelmer de Wolde <jelmer.de.wolde@alliander.com>

* Add support for alliander_gui.

Signed-off-by: Jelmer de Wolde <jelmer.de.wolde@alliander.com>

* Add option to start visualization for pytest.

Signed-off-by: Jelmer de Wolde <jelmer.de.wolde@alliander.com>

* Adapt pytest test_arm to support UR arm.

Signed-off-by: Jelmer de Wolde <jelmer.de.wolde@alliander.com>

* Prepare for hardware.

Signed-off-by: Jelmer de Wolde <jelmer.de.wolde@alliander.com>

* Moveit and joystick control on hardware.

Signed-off-by: Jelmer de Wolde <jelmer.de.wolde@alliander.com>

* Use arm in headless mode.

Signed-off-by: Jelmer de Wolde <jelmer.de.wolde@alliander.com>

* Add documentation.

Signed-off-by: Jelmer de Wolde <jelmer.de.wolde@alliander.com>

* Fix support for alliander_gui.

Signed-off-by: Jelmer de Wolde <jelmer.de.wolde@alliander.com>

* Fix linting.

Signed-off-by: Jelmer de Wolde <jelmer.de.wolde@alliander.com>

* Apply feedback.

Signed-off-by: Jelmer de Wolde <jelmer.de.wolde@alliander.com>

* Fix wave node for Franka.

Signed-off-by: Jelmer de Wolde <jelmer.de.wolde@alliander.com>

* Add functionality to unlock protective stop via dashboard.py and update docs

Signed-off-by: Rosalie <rosalie.van.ark@alliander.com>

* Fix wave demo for UR.

Signed-off-by: Jelmer de Wolde <jelmer.de.wolde@alliander.com>

* Fix linting.

Signed-off-by: Jelmer de Wolde <jelmer.de.wolde@alliander.com>

---------

Signed-off-by: Rosalie <rosalie.van.ark@alliander.com>
Signed-off-by: Jelmer de Wolde <jelmer.de.wolde@alliander.com>
Co-authored-by: Jelmer de Wolde <jelmer.de.wolde@alliander.com>
Co-authored-by: Jelmer de Wolde <Jelmerdw@users.noreply.github.com>

File: alliander_robotics/alliander_core/src/alliander_description/franka/urdf/adapted/franka_robot.xacro (robot description, xacro)
@@ -102,4 +102,10 @@
       />
     </xacro:if>
+    <!-- Add base_link: -->
+    <link name="base_link" />
+    <joint name="base_joint" type="fixed">
+      <parent link="base_link" />
+      <child  link="${arm_prefix}${arm_id}_link0" />
+    </joint>
     <!-- Definition of additional Gazebo tags -->
     <xacro:if value="${gazebo}">
@@ -112,5 +118,5 @@
           <origin xyz="${xyz}" rpy="${rpy}" />
           <parent link="${parent}" />
-          <child  link="${arm_prefix}${arm_id}_link0" />
+          <child  link="base_link" />
         </joint>
       </xacro:if>
