Commit message: Correct simulation specs.
Signed-off-by: Jelmer de Wolde <jelmer.de.wolde@alliander.com>

File: alliander_robotics/alliander_core/src/alliander_description/beamagine/urdf/l3cam.urdf.xacro (robot description, xacro)
@@ -4,6 +4,10 @@
 SPDX-License-Identifier: Apache-2.0
 -->
+<!--
+Specs based on:
+https://beamagine.com/wp-content/uploads/2022/05/DIGITAL-L3CAM-Robotic-vehicles-brochure.pdf
+https://github.com/beamaginelidar/l3cam_ros2
+-->
 <robot xmlns:xacro="http://www.ros.org/wiki/xacro" name="l3cam">
-  <xacro:property name="M_PI" value="3.1415926535897931" />
   <xacro:macro name="l3cam"
     params="
@@ -13,8 +17,4 @@
     lasers:=12
     samples:=1024
-    min_range:=0.5
-    max_range:=90.0
-    min_angle:=-${M_PI}
-    max_angle:=${M_PI}
     ">
     <!-- Gazebo requires a joint to a link called "world" for statically mounted robots -->
@@ -62,5 +62,5 @@
       <parent link="beamagine_camera_frame" />
       <child link="beamagine_camera_optical_frame" />
-      <origin xyz="0 0 0" rpy="-${M_PI/2} 0.0 -${M_PI/2}" />
+      <origin xyz="0 0 0" rpy="-${pi/2} 0.0 -${pi/2}" />
     </joint>
     <!-- Add gazebo plugin: -->
@@ -75,5 +75,4 @@
           <gz_frame_id>${namespace}/beamagine_camera_optical_frame</gz_frame_id>
           <camera>
-            <horizontal_fov>${110.0/180.0*pi}</horizontal_fov>
             <image>
               <width>640</width>
@@ -83,23 +82,4 @@
               <near>0.1</near>
               <far>300.0</far>
-            </clip>
-          </camera>
-        </sensor>
-        <!-- depth camera -->
-        <sensor type="depth_camera" name="beamagine_depth">
-          <always_on>true</always_on>
-          <update_rate>30.0</update_rate>
-          <topic>${namespace}/depth/image_rect_raw_float</topic>
-          <visualize>false</visualize>
-          <gz_frame_id>${namespace}/beamagine_camera_optical_frame</gz_frame_id>
-          <camera>
-            <horizontal_fov>${110.0/180.0*pi}</horizontal_fov>
-            <image>
-              <width>640</width>
-              <height>480</height>
-            </image>
-            <clip>
-              <near>0.2</near>
-              <far>65.536</far>
             </clip>
           </camera>
@@ -113,9 +93,7 @@
           <gz_frame_id>${namespace}/beamagine_camera_optical_frame</gz_frame_id>
           <camera>
-            <horizontal_fov>${58.0/180.0*pi}</horizontal_fov>
-            <vertical_fov>${42.0/180.0*pi}</vertical_fov>
             <image>
-              <width>320</width>
-              <height>240</height>
+              <width>640</width>
+              <height>480</height>
               <format>L16</format>
             </image>
@@ -147,18 +125,18 @@
                 <samples>${samples}</samples>
                 <resolution>1</resolution>
-                <min_angle>${min_angle}</min_angle>
-                <max_angle>${max_angle}</max_angle>
+                <min_angle>-${30/180*pi}</min_angle>
+                <max_angle> ${30/180*pi}</max_angle>
               </horizontal>
               <vertical>
                 <samples>${lasers}</samples>
                 <resolution>1</resolution>
-                <min_angle>-${21.2*M_PI/180.0}</min_angle>
-                <max_angle> ${21.2*M_PI/180.0}</max_angle>
+                <min_angle>-${10*pi/180.0}</min_angle>
+                <max_angle> ${10*pi/180.0}</max_angle>
               </vertical>
             </scan>
             <range>
-              <min>${min_range}</min>
-              <max>${max_range}</max>
-              <resolution>0.001</resolution>
+              <min>1.5</min>
+              <max>300.0</max>
+              <resolution>0.1</resolution>
             </range>
             <noise>
